File: Design/spudglo_driver_v4p1/spudglo_driver_v4p1.kicad_pcb (KiCad board)
At the start: 4 copper layers, 86.3 x 64.6 mm, 90 parts, among them J1 Barrel_Jack_Switch, J10 Conn_01x01_Male, J11 Conn_01x01_Male, J12 Conn_01x01_Male, J13 Conn_01x01_Male, J14 Conn_01x01_Male, J15 Conn_01x01_Male, J16 Conn_01x01_Male, J17 Conn_01x01_Male, J18 Conn_01x08_Male, J19 Conn_01x01_Male, J2 Conn_01x01_Male, J20 Conn_01x01_Male, J21 Conn_01x01_Male, J22 Conn_01x01_Male, J23 Conn_01x01_Male, J24 Conn_01x01_Male, J25 Conn_01x01_Male, J26 Conn_01x01_Male, J27 Conn_01x01_Male, J28 Conn_01x01_Male, J29 Conn_01x04_Male, J3 Conn_01x04_Male, J33 Conn_01x01_Male, J34 Conn_01x01_Male, J4 Conn_01x01_Male, J5 Conn_01x01_Male, J6 Conn_01x01_Male, J7 Conn_01x01_Male, J8 Conn_01x01_Male, J9 Conn_01x01_Male, SW1 SW_DIP_x01, U1 SN74HCT245PW, U10 receiver_433MHz, U11 receiver_433MHz, U2 STM32L431RCTx, U3 LP5907MFX-3.3, U4 ECS-480-8-36-RWN-TR, U5 receiver_433MHz, U6 ECS-.327-9-1210-TR, U7 PS2501-4, U8 TXB0104D, U9 receiver_433MHz

Commit message: schematic updates
Parts:
- removed C19: 1u, Capacitor_SMD:C_0603_1608Metric_Pad1.05x0.95mm_HandSolder
- removed J20, J21: Conn_01x01_Male, MountingHole:MountingHole_2.5mm_Pad
- U8: value TXB0104D -> TXS0104EDR
- moved R43 139.2 mm to (135.3, 84.6)
- moved R44 97.0 mm to (135.3, 98.1)
- moved U8 16.6 mm to (127.5, 107.3), turned to 90 degrees
- moved J3 14.3 mm to (140.9, 110.5)
- moved J1 8.55 mm to (136.1, 117.6)
- moved R30 5.24 mm to (135.3, 92.5)
- moved R29 4.44 mm to (135.3, 86.2)
- moved R34 4.21 mm to (135.3, 91.0), turned to 180 degrees
- moved R31 3.05 mm to (135.3, 89.4)
- moved R33 1.06 mm to (135.3, 87.8), turned to 180 degrees
- moved R40 0.28 mm to (135.3, 102.8)
- moved R41 0.17 mm to (135.3, 83.0)
- moved R42 0.11 mm to (135.3, 101.2)
- moved R35 0.08 mm to (135.3, 99.7)
Connections:
- net /Sheet62E58CB4/BOOT0 renamed /spudglo_driver_v4p1_micro/BOOT0
- net /Sheet62E58CB4/JTDI renamed /spudglo_driver_v4p1_micro/JTDI
- net /Sheet62E58CB4/JTDO renamed /spudglo_driver_v4p1_micro/JTDO
- net /Sheet62E58CB4/LVL_DIR renamed /spudglo_driver_v4p1_micro/LVL_DIR
- net /Sheet62E58CB4/LVL_EN renamed /spudglo_driver_v4p1_micro/LVL_EN
- net /Sheet62E58CB4/NJTRST renamed /spudglo_driver_v4p1_micro/NJTRST
- net /Sheet62E58CB4/NRST renamed /spudglo_driver_v4p1_micro/NRST
- net /Sheet62E58CB4/OSC48_HI renamed /spudglo_driver_v4p1_micro/OSC48_HI
- net /Sheet62E58CB4/OSC48_LO renamed /spudglo_driver_v4p1_micro/OSC48_LO
- net /Sheet62E58CB4/SWCLK renamed /spudglo_driver_v4p1_micro/SWCLK
- net /Sheet62E58CB4/SWDIO renamed /spudglo_driver_v4p1_micro/SWDIO
- net /Sheet62E58CB4/TIM15_CH1 renamed /spudglo_driver_v4p1_micro/TIM15_CH1
- net /Sheet62E58CB4/TIM15_CH1_SHIFT renamed /spudglo_driver_v4p1_micro/TIM15_CH1_SHIFT
- net /Sheet62E58CB4/TIM16_CH1 renamed /spudglo_driver_v4p1_micro/TIM16_CH1
- net /Sheet62E58CB4/TIM16_CH1_SHIFT renamed /spudglo_driver_v4p1_micro/TIM16_CH1_SHIFT
- net /Sheet62E58CB4/TIM1_CH1 renamed /spudglo_driver_v4p1_micro/TIM1_CH1
- net /Sheet62E58CB4/TIM1_CH1_SHIFT renamed /spudglo_driver_v4p1_micro/TIM1_CH1_SHIFT
- net /Sheet62E58CB4/TIM1_CH2 renamed /spudglo_driver_v4p1_micro/TIM1_CH2
- net /Sheet62E58CB4/TIM1_CH2_SHIFT renamed /spudglo_driver_v4p1_micro/TIM1_CH2_SHIFT
- net /Sheet62E58CB4/TIM1_CH3 renamed /spudglo_driver_v4p1_micro/TIM1_CH3
- net /Sheet62E58CB4/TIM1_CH3_SHIFT renamed /spudglo_driver_v4p1_micro/TIM1_CH3_SHIFT
- C18 pad 1: +3V3 -> +5V
Other:
- board text added: "5V+"

Commit message: spudglo_v4
Parts:
- removed C20: 1u, Capacitor_SMD:C_0603_1608Metric_Pad1.05x0.95mm_HandSolder
- removed J10, J11, J12, J14, J15, J16, J17, J19, J2, J22, J23, J24, J27, J28, J4, J5, J8, J9: Conn_01x01_Male, Connector_Pin:Pin_D1.3mm_L11.0mm
- removed J25, J26: Conn_01x01_Male, MountingHole:MountingHole_2.5mm_Pad
- removed J29: Conn_01x04_Male, Connector_PinHeader_2.54mm:PinHeader_1x04_P2.54mm_Vertical
- removed R27, R28: 100k, Resistor_SMD:R_0603_1608Metric_Pad1.05x0.95mm_HandSolder
- added C89: 1u, Capacitor_SMD:C_0603_1608Metric_Pad1.08x0.95mm_HandSolder, F.Cu at (123.6, 109.6)
- added G***: LOGO, LOGO, F.Cu at (158.8, 103.1)
- added G***: LOGO, LOGO, F.Cu at (152.5, 102.9)
- added G***: LOGO, LOGO, F.Cu at (165.2, 103.0)
- added REF**: WEEE-Logo_4.2x6mm_SilkScreen, Symbol:WEEE-Logo_4.2x6mm_SilkScreen, F.Cu at (149.5, 131.5)
- added REF**: ESD-Logo_6.6x6mm_SilkScreen, Symbol:ESD-Logo_6.6x6mm_SilkScreen, F.Cu at (178.3, 131.4)
- added REF**: RoHS-Logo_6mm_SilkScreen, Symbol:RoHS-Logo_6mm_SilkScreen, F.Cu at (163.4, 131.7)
- J13: value Conn_01x01_Male -> terminal_custom_9pin; footprint Connector_Pin:Pin_D1.3mm_L11.0mm -> Connector_Phoenix_MC:PhoenixContact_MCV_1,5_9-G-3.5_1x09_P3.50mm_Vertical
- J6, J7: footprint Connector_Pin:Pin_D1.3mm_L11.0mm -> MountingHole:MountingHole_2.5mm_Pad
- moved C18 148.0 mm to (123.6, 105.5), turned to -90 degrees
- moved C10 103.1 mm to (181.3, 116.9), turned to 180 degrees
- moved C11 102.6 mm to (175.5, 103.7), turned to 180 degrees
- moved C9 101.4 mm to (178.4, 115.1), turned to -90 degrees
- moved R39 95.3 mm to (135.0, 84.6), turned to 180 degrees
- moved C14 57.5 mm to (186.0, 126.4), turned to 0 degrees
- moved R13 57.3 mm to (184.4, 100.7), turned to -90 degrees
- moved SW1 55.6 mm to (174.6, 116.8)
- moved R9 54.1 mm to (187.5, 100.7), turned to -90 degrees
- moved J18 48.6 mm to (204.5, 84.0), turned to -90 degrees
- moved R5 37.6 mm to (194.2, 85.3), turned to 90 degrees
- moved R10 37.2 mm to (185.9, 100.7), turned to -90 degrees
- moved R8 36.6 mm to (189.1, 100.7)
- moved C21 35.5 mm to (189.1, 126.6), turned to 90 degrees
- moved R37 31.5 mm to (192.9, 105.0), turned to 0 degrees
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Connections:
- J13 pad 1: /spudglo_driver_v4p1_micro/TIM1_CH1_SHIFT -> +5V
- J3 pad 1: WKUP3 -> WKUP1
- J3 pad 2: WKUP4 -> WKUP2
- J3 pad 3: WKUP1 -> WKUP3
- J3 pad 4: WKUP2 -> WKUP4
- J7 pad 1: +5V -> GND1
- U1 pad 13: unconnected-(U1-Pad13) -> /spudglo_driver_v4p1_micro/TIM1_CH1_SHIFT
- U1 pad 14: /spudglo_driver_v4p1_micro/TIM15_CH1_SHIFT -> unconnected-(U1-Pad14)
- U1 pad 15: /spudglo_driver_v4p1_micro/TIM1_CH1_SHIFT -> /spudglo_driver_v4p1_micro/TIM1_CH2_SHIFT
- U1 pad 16: /spudglo_driver_v4p1_micro/TIM1_CH2_SHIFT -> unconnected-(U1-Pad16)
- U1 pad 18: /spudglo_driver_v4p1_micro/TIM16_CH1_SHIFT -> unconnected-(U1-Pad18)
- U1 pad 2: /spudglo_driver_v4p1_micro/TIM16_CH1 -> unconnected-(U1-Pad2)
- U1 pad 4: /spudglo_driver_v4p1_micro/TIM1_CH2 -> unconnected-(U1-Pad4)
- U1 pad 5: /spudglo_driver_v4p1_micro/TIM1_CH1 -> /spudglo_driver_v4p1_micro/TIM1_CH2
- U1 pad 6: /spudglo_driver_v4p1_micro/TIM15_CH1 -> unconnected-(U1-Pad6)
- U1 pad 7: unconnected-(U1-Pad7) -> /spudglo_driver_v4p1_micro/TIM1_CH1
- U2 pad 15: Net-(R27-Pad2) -> unconnected-(U2-Pad15)
- U2 pad 22: /spudglo_driver_v4p1_micro/TIM16_CH1 -> unconnected-(U2-Pad22)
- U2 pad 35: /spudglo_driver_v4p1_micro/TIM15_CH1 -> unconnected-(U2-Pad35)
Routing:
- net +3V3: track 0.00 -> 105.5 mm, vias 0 -> 12
- net /OUT_4_N: track 0.00 -> 85.0 mm
- net WKUP1: track 0.00 -> 68.4 mm, vias 0 -> 1
- net WKUP3: track 0.00 -> 67.1 mm, vias 0 -> 1
- net /OUT_3_N: track 0.00 -> 65.2 mm, vias 0 -> 1
- net WKUP2: track 0.00 -> 63.0 mm, vias 0 -> 1
- net /OUT_2_N: track 0.00 -> 61.9 mm
- net GND1: track 0.00 -> 59.8 mm, vias 0 -> 20
- net WKUP4: track 0.00 -> 59.3 mm, vias 0 -> 1
- net +5V: track 0.00 -> 56.7 mm, vias 0 -> 3
- net /OUT_4_P: track 0.00 -> 53.8 mm
- net /spudglo_driver_v4p1_micro/SWDIO: track 0.00 -> 53.0 mm, vias 0 -> 2
- net /spudglo_driver_v4p1_micro/NRST: track 0.00 -> 52.9 mm, vias 0 -> 2
- net /spudglo_driver_v4p1_micro/JTDI: track 0.00 -> 48.1 mm, vias 0 -> 2
- net /OUT_3_P: track 0.00 -> 43.3 mm, vias 0 -> 2
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Other:
- board text added: "01/18/2023 Spencer Wright Claire Drucker"
- board text added: "D1"
- board text added: "D2"
- board text added: "D3"
- board text added: "Facebook"
- board text added: "Instagram"
- board text added: "SpudGlo Driver 4.1 SpudGlo LLC www.SpudGlo.com"
- board text added: "SpudGlo.com"
- board text added: "WKUP1 (A)"
- board text added: "WKUP2 (B)"
- board text added: "WKUP3 (C)"
- board text added: "WKUP4 (D)"
- board text removed: "07/24/2022 Spencer Wright Claire Drucker"
- board text removed: "1"
- board text removed: "2"
- board text removed: "2022"
- board text removed: "3"
- board text removed: "3V3"
- board text removed: "4"
- board text removed: "5"
- board text removed: "INT_1"
- board text removed: "INT_2"
- board text removed: "INT_3"
- board text removed: "INT_4"
- board text removed: "J11"
- board text removed: "J12"
- board text removed: "J13"
- board text removed: "J17"
- board text removed: "J6"
- board text removed: "J7"
- board text removed: "JTDO"
- board text removed: "LED_2"
- board text removed: "NRST"
- board text removed: "SpudGlo Driver 3.1 SpudGlo LLC"
- board text removed: "WKUP3"
- board text removed: "WKUP4"

Commit message: spudglo v4p2!!!
Parts:
- removed the G*** at (158.8, 103.1)
- removed the G*** at (152.5, 102.9)
- removed the G*** at (165.2, 103.0)
- removed J13: terminal_custom_9pin, Connector_Phoenix_MC:PhoenixContact_MCV_1,5_9-G-3.5_1x09_P3.50mm_Vertical
- removed J33, J34, J6, J7: Conn_01x01_Male, MountingHole:MountingHole_2.5mm_Pad
- removed REF**: WEEE-Logo_4.2x6mm_SilkScreen, Symbol:WEEE-Logo_4.2x6mm_SilkScreen
- removed REF**: ESD-Logo_6.6x6mm_SilkScreen, Symbol:ESD-Logo_6.6x6mm_SilkScreen
- removed REF**: RoHS-Logo_6mm_SilkScreen, Symbol:RoHS-Logo_6mm_SilkScreen
- added F1: Fuse-2410FA, srw_custom:2410FA, F.Cu at (148.1, 127.3)
- added G***: LOGO, LOGO, F.Cu at (164.9, 124.9)
- added G***: LOGO, LOGO, F.Cu at (176.7, 124.8)
- added G***: LOGO, LOGO, F.Cu at (153.3, 124.9)
- added G***: LOGO, LOGO, F.Cu at (158.6, 109.2)
- added G***: LOGO, LOGO, B.Cu at (163.1, 87.7)
- added J2: terminal_custom_12pin, srw_custom:1984714, F.Cu at (204.0, 122.4)
- added R1: 10k, Resistor_SMD:R_0603_1608Metric_Pad0.98x0.95mm_HandSolder, F.Cu at (139.5, 113.7)
- moved R5 12.2 mm to (197.9, 96.9), turned to -90 degrees
- moved J18 10.3 mm to (197.7, 91.7), turned to 180 degrees
Connections:
- U2 pad 26: unconnected-(U2-Pad26) -> INT_LVL_EN
- U8 pad 8: +3V3 -> INT_LVL_EN
Routing:
- net INT_LVL_EN: track 0.00 -> 71.8 mm, vias 0 -> 2
- net GND1: track 59.8 -> 110.5 mm, vias 20 -> 24
- net +3V3: track 105.5 -> 132.1 mm, vias 12 -> 13
- net /spudglo_driver_v4p1_micro/NRST: track 52.9 -> 41.3 mm
- net /spudglo_driver_v4p1_micro/JTDI: track 48.1 -> 37.4 mm
- net /spudglo_driver_v4p1_micro/SWDIO: track 53.0 -> 42.7 mm
- net /spudglo_driver_v4p1_micro/NJTRST: track 40.3 -> 32.6 mm
- net /spudglo_driver_v4p1_micro/JTDO: track 36.0 -> 28.8 mm
- net +5V: track 56.7 -> 62.0 mm, vias 3 -> 4
- net Net-(J1-Pad1): track 31.9 -> 36.4 mm
- net /spudglo_driver_v4p1_micro/SWCLK: track 23.5 -> 21.0 mm
- net /spudglo_driver_v4p1_micro/TIM1_CH1_SHIFT: track 12.5 -> 10.7 mm
- net /spudglo_driver_v4p1_micro/TIM1_CH3_SHIFT: track 14.8 -> 13.5 mm
- net WKUP2: track 63.0 -> 64.0 mm
Other:
- board text added: "1A"
- board text added: "2B"
- board text added: "3C"
- board text added: "4D"
- board text removed: "WKUP1 (A)"
- board text removed: "WKUP2 (B)"
- board text removed: "WKUP3 (C)"
- board text removed: "WKUP4 (D)"
