File: Design/spudglo_driver_v4p1/spudglo_driver_v4p1.kicad_sch (KiCad schematic)
At the start: 20 parts, among them U10 receiver_433MHz, U11 receiver_433MHz, U5 receiver_433MHz, U7 PS2501-4, U8 TXB0104D, U9 receiver_433MHz

Commit message: schematic updates
Parts:
- removed C19: 1u, Capacitor_SMD:C_0603_1608Metric_Pad1.05x0.95mm_HandSolder, symbol Device:C_Small
- removed U8: TXB0104D, Package_SO:SOIC-14_3.9x8.7mm_P1.27mm, symbol Logic_LevelTranslator:TXB0104D
- added C5: 1u, Capacitor_SMD:C_0603_1608Metric_Pad1.05x0.95mm_HandSolder, symbol Device:C_Small
- added U8: TXS0104EDR, Package_SO:SOIC-14_3.9x8.7mm_P1.27mm, symbol srw_custom:TXS0104EDR
Connections:
- net +3V3: now also C5.1, U8.1 (VCCA), U8.8 (OE); no longer C18.1
- net +5V: now also C18.1, U8.14 (VCCB)
- net GND1: now also C5.2, U8.7 (GND)
- net INT_1: now also U8.13 (B1)
- net INT_2: now also U8.12 (B2)
- net INT_3: now also U8.11 (B3)
- net INT_4: now also U8.10 (B4)
- net WKUP1: now also U8.2 (A1)
- net WKUP2: now also U8.3 (A2)
- net WKUP3: now also U8.4 (A3)
- net WKUP4: now also U8.5 (A4)
- no-connect marks 4 -> 6
Other:
- removed sheet Sheet62E58CB4
- added sheet spudglo_driver_v4p1_micro (spudglo_driver_v4p1_micro.kicad_sch)

Commit message: spudglo_v4
Parts:
- removed C5: 1u, Capacitor_SMD:C_0603_1608Metric_Pad1.05x0.95mm_HandSolder, symbol Device:C_Small
- added C89: 1u, Capacitor_SMD:C_0603_1608Metric_Pad1.08x0.95mm_HandSolder, symbol Device:C_Small
Connections:
- net +3V3: now also C89.1
- net GND1: now also C89.2

Commit message: spudglo v4p2!!!
Parts:
- added R1: 10k, Resistor_SMD:R_0603_1608Metric_Pad0.98x0.95mm_HandSolder, symbol Device:R
Connections:
- net +3V3: no longer U8.8 (OE)
- net GND1: now also R1.2
- new net INT_LVL_EN: R1.1, U8.8 (OE)
Other:
- moved on the sheet: C89
