File: Design/spudglo_driver_v4p1/spudglo_driver_v4p1_micro.kicad_sch (KiCad schematic)
At the start: 20 parts, among them U10 receiver_433MHz, U11 receiver_433MHz, U5 receiver_433MHz, U7 PS2501-4, U8 TXB0104D, U9 receiver_433MHz

Commit message: schematic updates
Parts:
- removed C18, C19: 1u, Capacitor_SMD:C_0603_1608Metric_Pad1.05x0.95mm_HandSolder, symbol Device:C_Small
- removed R29, R30, R41, R42: 1k, Resistor_SMD:R_0603_1608Metric_Pad1.05x0.95mm_HandSolder, symbol Device:R
- removed R31, R33, R34, R35, R39, R40, R43, R44: 10k, Resistor_SMD:R_0603_1608Metric_Pad1.05x0.95mm_HandSolder, symbol Device:R
- removed U10, U11, U5, U9: receiver_433MHz, Connector_PinHeader_2.54mm:PinHeader_1x05_P2.54mm_Vertical, symbol spudglo_driver_v3p1-rescue:receiver_433MHz-srw_custom
- removed U7: PS2501-4, Package_DIP:DIP-16_W7.62mm_LongPads, symbol spudglo_driver_v3p1-rescue:PS2501-4-srw_custom
- removed U8: TXB0104D, Package_SO:SOIC-14_3.9x8.7mm_P1.27mm, symbol Logic_LevelTranslator:TXB0104D
- added C1, C2: 6p, Capacitor_SMD:C_0603_1608Metric_Pad1.05x0.95mm_HandSolder, symbol spudglo_driver_v3p1-rescue:CP_Small-Device
- added C10, C11, C12, C6, C7, C8, C9: 0.1u, Capacitor_SMD:C_0603_1608Metric_Pad1.05x0.95mm_HandSolder, symbol spudglo_driver_v3p1-rescue:CP_Small-Device
- added C13: 4.7u, Capacitor_SMD:C_0603_1608Metric_Pad1.05x0.95mm_HandSolder, symbol spudglo_driver_v3p1-rescue:CP_Small-Device
- added C14, C17, C20: 1u, Capacitor_SMD:C_0603_1608Metric_Pad1.05x0.95mm_HandSolder, symbol spudglo_driver_v3p1-rescue:CP_Small-Device
- added C15: 0.01u, Capacitor_SMD:C_0603_1608Metric_Pad1.05x0.95mm_HandSolder, symbol spudglo_driver_v3p1-rescue:CP_Small-Device
- added C16: 1, Capacitor_SMD:C_0603_1608Metric_Pad1.05x0.95mm_HandSolder, symbol spudglo_driver_v3p1-rescue:CP_Small-Device
- added C21: 10u, Capacitor_SMD:C_0603_1608Metric_Pad1.05x0.95mm_HandSolder, symbol spudglo_driver_v3p1-rescue:CP_Small-Device
- added C3, C4: 8p, Capacitor_SMD:C_0603_1608Metric_Pad1.05x0.95mm_HandSolder, symbol spudglo_driver_v3p1-rescue:CP_Small-Device
- added H1, H2, H3, H4: MountingHole, MountingHole:MountingHole_6.5mm, symbol Mechanical:MountingHole
- added J1: Barrel_Jack_Switch, Connector_BarrelJack:BarrelJack_Wuerth_6941xx301002, symbol Connector:Barrel_Jack_Switch
- added J10, J11, J12, J13, J14, J15, J16, J17, J19, J2, J22, J23, J24, J27, J28, J4, J5, J6, J7, J8, J9: Conn_01x01_Male, Connector_Pin:Pin_D1.3mm_L11.0mm, symbol Connector:Conn_01x01_Male
- added J18: Conn_01x08_Male, Connector_PinHeader_2.54mm:PinHeader_2x04_P2.54mm_Vertical, symbol Connector:Conn_01x08_Male
- added J25, J26, J33, J34: Conn_01x01_Male, MountingHole:MountingHole_2.5mm_Pad, symbol Connector:Conn_01x01_Male
- added J29, J3: Conn_01x04_Male, Connector_PinHeader_2.54mm:PinHeader_1x04_P2.54mm_Vertical, symbol Connector:Conn_01x04_Male
- added R10, R13, R2, R3, R37, R38, R5, R8, R9: 10k, Resistor_SMD:R_0603_1608Metric_Pad1.05x0.95mm_HandSolder, symbol Device:R
- added R27, R28: 100k, Resistor_SMD:R_0603_1608Metric_Pad1.05x0.95mm_HandSolder, symbol Device:R
- added SW1: SW_DIP_x01, Connector_PinHeader_2.54mm:PinHeader_1x02_P2.54mm_Vertical, symbol Switch:SW_DIP_x01
- added U1: SN74HCT245PW, Package_SO:TSSOP-20_4.4x6.5mm_P0.65mm, symbol spudglo_driver_v3p1-rescue:SN74HCT245PW-srw_custom
- added U2: STM32L431RCTx, Package_QFP:LQFP-64_10x10mm_P0.5mm, symbol spudglo_driver_v3p1-rescue:STM32L431RCTx-MCU_ST_STM32L4
- added U3: LP5907MFX-3.3, Package_TO_SOT_SMD:SOT-23-5, symbol Regulator_Linear:LP5907MFX-3.3
- added U4: ECS-480-8-36-RWN-TR, XTAL_ECS-480-8-36-RWN-TR, symbol spudglo_driver_v3p1-rescue:ECS-480-8-36-RWN-TR-ECS-480-8-36-RWN-TR
- added U6: ECS-.327-9-1210-TR, ECS-:XTAL_ECS-.327-9-1210-TR, symbol Device:Crystal
Connections:
- net +3V3: now also C10.1, C11.1, C12.1, C13.1, C15.1, C16.1, C17.1, C20.1, C8.1, C9.1, J18.8 (Pin_8), J2.1 (Pin_1), J29.2 (Pin_2), R10.1, R13.1, R27.1, R3.1, R37.1, R5.1, R8.1, R9.1, U2.1 (VBAT), U2.13 (VDDA), U2.19 (VDD), U2.32 (VDD), U2.48 (VDDUSB), U2.64 (VDD), U3.5 (OUT)
- net +5V: now also C14.1, C21.1, C7.1, J14.1 (Pin_1), J15.1 (Pin_1), J25.1 (Pin_1), J27.1 (Pin_1), J29.4 (Pin_4), J34.1 (Pin_1), J5.1 (Pin_1), J6.1 (Pin_1), J7.1 (Pin_1), J8.1 (Pin_1), U1.20 (VCC), U3.1 (IN), U3.3 (EN)
- net GND1: now also C1.2, C10.2, C11.2, C12.2, C13.2, C14.2, C15.2, C16.2, C17.2, C2.2, C20.2, C21.2, C3.2, C4.2, C6.2, C7.2, C8.2, C9.2, J1.2, J1.3, J10.1 (Pin_1), J11.1 (Pin_1), J12.1 (Pin_1), J16.1 (Pin_1), J18.1 (Pin_1), J24.1 (Pin_1), J26.1 (Pin_1), J28.1 (Pin_1), J29.1 (Pin_1), J29.3 (Pin_3), J4.1 (Pin_1), J9.1 (Pin_1), R2.2, R28.2, R38.2, SW1.2, U1.10 (GND), U2.12 (VSSA), U2.18 (VSS), U2.31 (VSS), U2.47 (VSS), U2.63 (VSS), U3.2 (GND), U4.2 (GND), U4.4 (GND)
- net WKUP1: now also J3.3 (Pin_3), U2.14 (PA0_WKUP1)
- net WKUP2: now also J3.4 (Pin_4), U2.2 (PC13/WKUP2)
- net WKUP3: now also J3.1 (Pin_1), U2.25 (PC5/USART3_RX/WKUP5)
- net WKUP4: now also J3.2 (Pin_2), U2.16 (PA2/LPUART1_TX/TIM2_CH3/WKUP4)
- new net: R27.2, R28.1, U2.15 (PA1_SPI1_SCK)
- new net: C4.1, U2.3 (PC14_OSC32_IN), U6.1
- new net: C3.1, U2.4 (PC15_OSC32_OUT), U6.2
- new net: J1.1, J33.1 (Pin_1)
- new net BOOT0: R2.1, U2.60 (PH3/BOOT0)
- new net JTDI: J18.5 (Pin_5), R9.2, U2.50 (PA15/JTDI)
- new net JTDO: J18.4 (Pin_4), R10.2, U2.55 (PB3/JTDO-TRACE-SWO)
- new net LVL_DIR: R37.2, U1.1 (DIR), U2.39 (PC8)
- new net LVL_EN: R38.1, U1.19 (OE_N), U2.38 (PC7)
- new net NJTRST: J18.3 (Pin_3), R13.2, U2.56 (PB4/NJTRST)
- new net NRST: C6.1, J18.2 (Pin_2), R3.2, SW1.1, U2.7 (NRST)
- new net OSC48_HI: C2.1, U2.5 (PH0/OSCIN), U4.3 (OUT/IN)
- new net OSC48_LO: C1.1, U2.6 (PH1/OSCOUT), U4.1 (IN/OUT)
- new net SWCLK: J18.6 (Pin_6), R8.2, U2.49 (PA14/SWCLK)
- new net SWDIO: J18.7 (Pin_7), R5.2, U2.46 (PA13/SWDIO)
- new net TIM15_CH1: U1.6 (A5), U2.35 (PB14/SPI2_MISO/TIM15_CH1)
- new net TIM15_CH1_SHIFT: J22.1 (Pin_1), U1.14 (B5)
- new net TIM16_CH1: U1.2 (A1), U2.22 (PA6/TIM16_CH1)
- new net TIM16_CH1_SHIFT: J23.1 (Pin_1), U1.18 (B1)
- new net TIM1_CH1: U1.5 (A4), U2.41 (PA8/TIM1_CH1)
- new net TIM1_CH1_SHIFT: J13.1 (Pin_1), U1.15 (B4)
- new net TIM1_CH2: U1.4 (A3), U2.42 (PA9/TIM1_CH2/USART1_TX)
- new net TIM1_CH2_SHIFT: J17.1 (Pin_1), U1.16 (B3)
- new net TIM1_CH3: U1.3 (A2), U2.43 (PA10/TIM1_CH3/USART1_RX)
- new net TIM1_CH3_SHIFT: J19.1 (Pin_1), U1.17 (B2)
- no-connect marks 4 -> 36
Other:
- removed sheet Sheet62E58CB4

Commit message: spudglo_v4
Parts:
- removed C20: 1u, Capacitor_SMD:C_0603_1608Metric_Pad1.05x0.95mm_HandSolder, symbol spudglo_driver_v3p1-rescue:CP_Small-Device
- removed J10, J11, J12, J13, J14, J15, J16, J17, J19, J2, J22, J23, J24, J27, J28, J4, J5, J8, J9: Conn_01x01_Male, Connector_Pin:Pin_D1.3mm_L11.0mm, symbol Connector:Conn_01x01_Male
- removed J25, J26: Conn_01x01_Male, MountingHole:MountingHole_2.5mm_Pad, symbol Connector:Conn_01x01_Male
- removed J29: Conn_01x04_Male, Connector_PinHeader_2.54mm:PinHeader_1x04_P2.54mm_Vertical, symbol Connector:Conn_01x04_Male
- removed R27, R28: 100k, Resistor_SMD:R_0603_1608Metric_Pad1.05x0.95mm_HandSolder, symbol Device:R
- added J13: terminal_custom_9pin, Connector_Phoenix_MC:PhoenixContact_MCV_1,5_9-G-3.5_1x09_P3.50mm_Vertical, symbol srw_custom:terminal_custom_9pin
- J6, J7: footprint Connector_Pin:Pin_D1.3mm_L11.0mm -> MountingHole:MountingHole_2.5mm_Pad
Connections:
- net +5V: now also J13.1, J13.4, J13.7; no longer J7.1 (Pin_1)
- net GND1: now also J7.1 (Pin_1), J13.3, J13.6, J13.9
- net TIM1_CH1: now also U1.7 (A6); no longer U1.5 (A4)
- net TIM1_CH1_SHIFT: now also U1.13 (B6), J13.2; no longer U1.15 (B4)
- net TIM1_CH2: now also U1.5 (A4); no longer U1.4 (A3)
- net TIM1_CH2_SHIFT: now also U1.15 (B4), J13.5; no longer U1.16 (B3)
- net TIM1_CH3_SHIFT: now also J13.8
- net WKUP1: now also J3.1 (Pin_1); no longer J3.3 (Pin_3)
- net WKUP2: now also J3.2 (Pin_2); no longer J3.4 (Pin_4)
- net WKUP3: now also J3.3 (Pin_3); no longer J3.1 (Pin_1)
- net WKUP4: now also J3.4 (Pin_4); no longer J3.2 (Pin_2)
- net TIM15_CH1: no longer names the net of U2.35 (PB14/SPI2_MISO/TIM15_CH1)
- net TIM15_CH1: no longer U1.6 (A5)
- net TIM15_CH1_SHIFT: no longer names the net of U1.14 (B5)
- net TIM16_CH1: no longer names the net of U2.22 (PA6/TIM16_CH1)
- net TIM16_CH1: no longer U1.2 (A1)
- net TIM16_CH1_SHIFT: no longer names the net of U1.18 (B1)
- no-connect marks 36 -> 44

Commit message: spudglo v4p2!!!
Parts:
- removed J13: terminal_custom_9pin, Connector_Phoenix_MC:PhoenixContact_MCV_1,5_9-G-3.5_1x09_P3.50mm_Vertical, symbol srw_custom:terminal_custom_9pin
- removed J33, J34, J6, J7: Conn_01x01_Male, MountingHole:MountingHole_2.5mm_Pad, symbol Connector:Conn_01x01_Male
- added F1: Fuse-2410FA, srw_custom:2410FA, symbol srw_custom:Fuse-2410FA
- added J2: terminal_custom_12pin, srw_custom:1984714, symbol srw_custom:terminal_custom_12pin
Connections:
- net +5V: now also F1.2, J2.1, J2.10, J2.4, J2.7
- net GND1: now also J2.12, J2.3, J2.6, J2.9
- net TIM1_CH1_SHIFT: now also J2.2
- net TIM1_CH2_SHIFT: now also J2.5
- net TIM1_CH3_SHIFT: now also J2.8
- net INT_LVL_EN: now reaches U2.26 (PB0)
- net at J1.1: now also F1.1
- no-connect marks 44 -> 45
