File: Design/spudglo_driver_v4p2/spudglo_driver_v4p2/spudglo_driver_v4p2.kicad_pcb (KiCad board)
At the start: 4 copper layers, 65 x 39 mm, 61 parts, among them J1 locked, J2 Barrel_Jack_Switch, U1 receiver_433MHz, U10 STM32L431RCTx, U11 LP5907MFX-3.3, U2 TXS0104EDR, U3 receiver_433MHz, U4 receiver_433MHz, U5 receiver_433MHz, U6 PS2501-4, U7 ECS-.327-9-1210-TR, U8 ECS-480-8-36-RWN-TR, U9 SN74HCT245PW

Commit message: usb add
Parts:
- added C20: 1u, Capacitor_SMD:C_0603_1608Metric_Pad1.08x0.95mm_HandSolder, F.Cu at (257.0, 27.1)
- added C21: 1u, Capacitor_SMD:C_0603_1608Metric_Pad1.08x0.95mm_HandSolder, F.Cu at (255.6, 17.0)
- added C22: 1u, Capacitor_SMD:C_0603_1608Metric_Pad1.08x0.95mm_HandSolder, F.Cu at (252.7, 30.0)
- added C23: 1u, Capacitor_SMD:C_0603_1608Metric_Pad1.08x0.95mm_HandSolder, F.Cu at (260.0, 24.6)
- added C24: 0.1u, Capacitor_SMD:C_0603_1608Metric_Pad1.08x0.95mm_HandSolder, F.Cu at (264.3, 17.0)
- added C25: 1u, Capacitor_SMD:C_0603_1608Metric_Pad1.08x0.95mm_HandSolder, F.Cu at (260.0, 17.0)
- added C26: 1u, Capacitor_SMD:C_0603_1608Metric_Pad1.08x0.95mm_HandSolder, F.Cu at (264.3, 22.1)
- added R25: 5.1k, Resistor_SMD:R_0603_1608Metric_Pad0.98x0.95mm_HandSolder, F.Cu at (248.3, 27.5)
- added R26: 5.1k, Resistor_SMD:R_0603_1608Metric_Pad0.98x0.95mm_HandSolder, F.Cu at (255.6, 24.6)
- added R27: 0, Resistor_SMD:R_0603_1608Metric_Pad0.98x0.95mm_HandSolder, F.Cu at (252.7, 27.5)
- added R28: 0, Resistor_SMD:R_0603_1608Metric_Pad0.98x0.95mm_HandSolder, F.Cu at (255.6, 22.1)
- added R29: 0, Resistor_SMD:R_0603_1608Metric_Pad0.98x0.95mm_HandSolder, F.Cu at (255.6, 19.6)
- added R30: 0, Resistor_SMD:R_0603_1608Metric_Pad0.98x0.95mm_HandSolder, F.Cu at (248.3, 30.0)
- added R31: 0, Resistor_SMD:R_0603_1608Metric_Pad0.98x0.95mm_HandSolder, F.Cu at (260.0, 22.1)
- added R32: 10k, Resistor_SMD:R_0603_1608Metric_Pad0.98x0.95mm_HandSolder, F.Cu at (264.3, 19.6)
- added R33: 10k, Resistor_SMD:R_0603_1608Metric_Pad0.98x0.95mm_HandSolder, F.Cu at (260.0, 19.6)
- added U12: USB-C-31-M-12, Connector_USB:USB_C_Receptacle_HRO_TYPE-C-31-M-12, F.Cu at (247.6, 21.6)
- added U13: XR21B1411, srw_custom:XR21B1411, F.Cu at (242.6, 27.7)
Connections:
- net /spudglo_v4p2_micro/NRST renamed NRST
- U10 pad 10: unconnected-(U10-Pad10) -> XR_GPIO
- U10 pad 8: unconnected-(U10-Pad8) -> XR_TX
- U10 pad 9: unconnected-(U10-Pad9) -> XR_RX
Routing:
- net WKUP2: track 61.3 -> 56.5 mm
Other:
- board text removed: "receiver_433MHz"
