File: Design/spudglo_driver_v4p2/spudglo_driver_v4p2/spudglo_driver_v4p2.kicad_sch (KiCad schematic)
At the start: 22 parts, among them U1 receiver_433MHz, U2 TXS0104EDR, U3 receiver_433MHz, U4 receiver_433MHz, U5 receiver_433MHz, U6 PS2501-4

Commit message: more hw lol
Parts:
- U6: footprint Package_DIP:DIP-16_W7.62mm_LongPads -> srw_custom:PS2501-4XSM
Connections:
- net INT_1: now also U2.10 (B4); no longer U2.13 (B1)
- net INT_2: now also U2.11 (B3); no longer U2.12 (B2)
- net INT_3: now also U2.12 (B2); no longer U2.11 (B3)
- net INT_4: now also U2.13 (B1); no longer U2.10 (B4)
Changed lines of the file:
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@@
     (stroke (width 0) (type default) (color 0 0 0 0))
   )
-  (label "INT_2" (at 90.17 123.19 0)
+  (label "INT_3" (at 90.17 123.19 0)
     (effects (font (size 1.27 1.27)) (justify left bottom))
   )
@@
     (effects (font (size 1.27 1.27)) (justify right bottom))
   )
-  (label "INT_1" (at 90.17 120.65 0)
+  (label "INT_4" (at 90.17 120.65 0)
     (effects (font (size 1.27 1.27)) (justify left bottom))
   )
@@
     (effects (font (size 1.27 1.27)) (justify right bottom))
   )
-  (label "INT_3" (at 90.17 125.73 0)
+  (label "INT_2" (at 90.17 125.73 0)
     (effects (font (size 1.27 1.27)) (justify left bottom))
   )
@@
     (effects (font (size 1.27 1.27)) (justify right bottom))
   )
-  (label "INT_4" (at 90.17 128.27 0)
+  (label "INT_1" (at 90.17 128.27 0)
     (effects (font (size 1.27 1.27)) (justify left bottom))
   )
@@
     (property "Reference" "U6" (id 0) (at 207.645 112.649 0))
     (property "Value" "PS2501-4" (id 1) (at 207.645 114.9604 0))
-    (property "Footprint" "Package_DIP:DIP-16_W7.62mm_LongPads" (id 2) (at 194.31 114.3 0)
+    (property "Footprint" "srw_custom:PS2501-4XSM" (id 2) (at 194.31 114.3 0)
       (effects (font (size 1.27 1.27)) hide)
     )
@@
       (reference "J4") (unit 1) (value "Conn_01x08_Male") (footprint "Connector_PinHeader_2.54mm:PinHeader_1x08_P2.54mm_Vertical")
     )
+    (path "/5af74bf5-987c-4d46-98f6-b35b1497740a/7438c70b-8a8f-4566-b08c-1dd2215ef48a"
+      (reference "J5") (unit 1) (value "Conn_01x02_Male") (footprint "Connector_PinHeader_2.54mm:PinHeader_1x02_P2.54mm_Vertical")
+    )
     (path "/5af74bf5-987c-4d46-98f6-b35b1497740a/295cc4b7-6c68-450f-8cf9-bf7a423e9350"
       (reference "MH1") (unit 1) (value "MountingHole_Pad") (footprint "MountingHole:MountingHole_3mm")
@@
       (reference "MH2") (unit 1) (value "MountingHole_Pad") (footprint "MountingHole:MountingHole_3mm")
     )
-    (path "/5af74bf5-987c-4d46-98f6-b35b1497740a/e8594e03-7d6e-4a74-8a55-664d2faab756"
-      (reference "MH3") (unit 1) (value "MountingHole_Pad") (footprint "MountingHole:MountingHole_3mm")
-    )
-    (path "/5af74bf5-987c-4d46-98f6-b35b1497740a/1a8efcec-8d90-47a7-9f35-3a7ff2204492"
-      (reference "MH4") (unit 1) (value "MountingHole_Pad") (footprint "MountingHole:MountingHole_3mm")
-    )
     (path "/bc7bb465-968b-4df0-91f2-2cdf51749f16"
       (reference "R1") (unit 1) (value "10k") (footprint "Resistor_SMD:R_0603_1608Metric_Pad0.98x0.95mm_HandSolder")
@@
     )
     (path "/314b6d97-8942-4f04-b778-5e452d16f1c6"
-      (reference "U6") (unit 1) (value "PS2501-4") (footprint "Package_DIP:DIP-16_W7.62mm_LongPads")
+      (reference "U6") (unit 1) (value "PS2501-4") (footprint "srw_custom:PS2501-4XSM")
     )
     (path "/5af74bf5-987c-4d46-98f6-b35b1497740a/75f32061-e5ce-46df-82c2-a58776da8ca7"
