File: Design/spudglo_driver_v4p2/spudglo_driver_v4p2/spudglo_v4p2_micro.kicad_sch (KiCad schematic)
At the start: 36 parts, among them J1 Conn_01x08_Male, J2 Barrel_Jack_Switch, J3 terminal_custom_12pin, U10 STM32L431RCTx, U11 LP5907MFX-3.3, U7 ECS-.327-9-1210-TR, U8 ECS-480-8-36-RWN-TR, U9 SN74HCT245PW

Commit message: usb add
Parts:
- added C20, C21, C22, C23, C25, C26: 1u, Capacitor_SMD:C_0603_1608Metric_Pad1.08x0.95mm_HandSolder, symbol spudglo_driver_v3p1-rescue:CP_Small-Device
- added C24: 0.1u, Capacitor_SMD:C_0603_1608Metric_Pad1.08x0.95mm_HandSolder, symbol spudglo_driver_v3p1-rescue:CP_Small-Device
- added R25, R26: 5.1k, Resistor_SMD:R_0603_1608Metric_Pad0.98x0.95mm_HandSolder, symbol Device:R
- added R27, R28, R29, R30, R31: 0, Resistor_SMD:R_0603_1608Metric_Pad0.98x0.95mm_HandSolder, symbol Device:R
- added R32, R33, R?: 10k, Resistor_SMD:R_0603_1608Metric_Pad0.98x0.95mm_HandSolder, symbol Device:R
- added R?: 28k, Resistor_SMD:R_0603_1608Metric_Pad0.98x0.95mm_HandSolder, symbol Device:R
- added U12: USB-C-31-M-12, Connector_USB:USB_C_Receptacle_HRO_TYPE-C-31-M-12, symbol srw_custom:USB-C-31-M-12
- added U?: XR21B1411, srw_custom:XR21B1411, symbol srw_custom:XR21B1411
Connections:
- net +3V3: now also C20.1, C21.1, C22.1, C23.1, C25.1, C26.1, R31.1, R?.1, U12.A4 (VBUS4), U12.A9 (VBUS1), U12.B4 (VBUS3), U12.B9 (VBUS2), U?.12 (VIO_REF), U?.16 (VCC)
- net GND1: now also C20.2, C21.2, C22.2, C23.2, C24.2, C25.2, C26.2, R25.2, R26.2, R32.2, R33.2, R?.2, U12.A1 (GND2), U12.A12 (GND4), U12.B1 (GND1), U12.B12 (GND3), U?.13 (GND1), U?.EPAD (GND2)
- net INT_LVL_EN: now also R30.1
- net NRST: now also R27.1
- net WKUP1: now also R28.1
- net XR_GPIO: now reaches U10.10 (PC2/SPI2_MISO)
- net XR_GPIO: now also R29.1
- net VBUS_PRESENT: now reaches U10.17 (PA3/LPUART1_RX/TIM2_CH4)
- net VBUS_PRESENT: now also R?.1, R?.2
- net XR_TX: now reaches U10.8 (PC0/LPUART1_RX)
- net XR_TX: now also U?.9 (TX)
- net XR_RX: now reaches U10.9 (PC1/LPUART1_TX)
- net XR_RX: now also U?.10 (RX)
- new net: R26.1, U12.A5 (CC1)
- new net: R25.1, U12.B5 (CC2)
- new net: R29.2, U?.6 (GPIO2)
- new net: R28.2, U?.7 (GPIO1)
- new net: R33.1, U?.1 (LOWPOWER)
- new net: R30.2, U?.5 (GPIO3)
- new net: R27.2, U?.8 (GPIO0)
- new net: C24.1, R31.2, R32.1, U?.11 (VBUS_SENSE)
- new net USBD+: U12.A6 (DP1), U12.B6 (DP2), U?.15 (USBD+)
- new net USBD-: U12.A7 (DN1), U12.B7 (DN2), U?.14 (USBD-)
- no-connect marks 44 -> 45
Other:
- moved on the sheet: J3

Commit message: spudglo_driver_v4p2_final
Parts:
- removed C20, C21, C22, C23: 1u, Capacitor_SMD:C_0603_1608Metric_Pad1.08x0.95mm_HandSolder, symbol spudglo_driver_v3p1-rescue:CP_Small-Device
- removed C24: 0.1u, Capacitor_SMD:C_0603_1608Metric_Pad1.08x0.95mm_HandSolder, symbol spudglo_driver_v3p1-rescue:CP_Small-Device
- added C27, C28: 1u, Capacitor_SMD:C_0603_1608Metric_Pad1.08x0.95mm_HandSolder, symbol spudglo_driver_v3p1-rescue:CP_Small-Device
- added J4: Conn_01x08_Male, Connector_PinHeader_2.54mm:PinHeader_1x08_P2.54mm_Vertical, symbol Connector:Conn_01x08_Male
- added MH1, MH2, MH3, MH4: MountingHole_Pad, MountingHole:MountingHole_3mm, symbol Mechanical:MountingHole_Pad
- added R36: 10k, Resistor_SMD:R_0603_1608Metric_Pad0.98x0.95mm_HandSolder, symbol Device:R
- added U14: NCP361, srw_custom:NCP361, symbol srw_custom:NCP361
- R32: value 10k -> DNI
- gave numbers to parts that had none: 3
Connections:
- net +3V3: now also J4.2 (Pin_2), R36.1; no longer C26.1, R31.1, R34.1, U12.A4 (VBUS4), U12.A9 (VBUS1), U12.B4 (VBUS3), U12.B9 (VBUS2), U13.16 (VCC)
- net GND1: now also C27.2, C28.2, J4.1 (Pin_1), MH1.1, MH2.1, MH3.1, MH4.1, U14.1 (EN_N), U14.2 (GND1), U14.EPAD (GND2); no longer R32.2
- net VBUS_PRESENT: now also U10.34 (PB13); no longer U10.17 (PA3/LPUART1_RX/TIM2_CH4)
- net XR_GPIO: now also U10.33 (PB12); no longer U10.10 (PC2/SPI2_MISO)
- net XR_RX: now also U10.58 (PB6/USART1_TX); no longer U10.9 (PC1/LPUART1_TX)
- net XR_TX: now also U10.59 (PB7/USART1_RX); no longer U10.8 (PC0/LPUART1_RX)
- net SPI1_SCK: now reaches U10.15 (PA1_SPI1_SCK)
- net SPI1_SCK: now also J4.3 (Pin_3)
- net SPI1_NSS: now reaches U10.20 (PA4/SPI1_NSS/LPTIM2_OUT)
- net SPI1_NSS: now also J4.7 (Pin_7), R36.2
- net DISP_BACKLIGHT: now reaches U10.21 (PA5/SPI1_SCK/TIM2_CH1)
- net DISP_BACKLIGHT: now also J4.8 (Pin_8)
- net DISP_DC: now reaches U10.22 (PA6/TIM16_CH1)
- net DISP_DC: now also J4.6 (Pin_6)
- net DISP_RST: now reaches U10.23 (PA7/SPI1_MOSI)
- net DISP_RST: now also J4.5 (Pin_5)
- net SPI1_CIPO: now reaches U10.44 (PA11/TIM1_CH4/SPI1_MISO)
- net SPI1_CIPO: now also R32.1
- net SPI1_COPI: now reaches U10.45 (PA12/SPI_MOSI)
- net SPI1_COPI: now also R31.1
- new net: C27.1, U12.A4 (VBUS4), U12.A9 (VBUS1), U12.B4 (VBUS3), U12.B9 (VBUS2), U14.3 (IN)
- new net: J4.4 (Pin_4), R31.2, R32.2
- new net VBUS: C26.1, C28.1, R34.1, U13.16 (VCC), U14.4 (OUT1), U14.5 (OUT2)
- now unconnected: U13.11 (VBUS_SENSE)
- no-connect marks 45 -> 38
Other:
- moved on the sheet: J3

Commit message: more hw lol
Parts:
- removed MH3, MH4: MountingHole_Pad, MountingHole:MountingHole_3mm, symbol Mechanical:MountingHole_Pad
- added J5: Conn_01x02_Male, Connector_PinHeader_2.54mm:PinHeader_1x02_P2.54mm_Vertical, symbol Connector:Conn_01x02_Male
Connections:
- net GND1: now also U13.11 (VBUS_SENSE)
- net XR_RX: now also U10.9 (PC1/LPUART1_TX); no longer U10.58 (PB6/USART1_TX)
- net XR_TX: now also U10.8 (PC0/LPUART1_RX); no longer U10.59 (PB7/USART1_RX)
- no-connect marks 38 -> 37
Changed lines of the file:
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@@
   (junction (at 274.32 44.45) (diameter 0) (color 0 0 0 0)
   )
+  (junction (at 194.31 52.07) (diameter 0) (color 0 0 0 0)
+  )
   (junction (at 205.74 147.32) (diameter 0) (color 0 0 0 0)
   )
@@
   (junction (at 177.8 110.49) (diameter 0) (color 0 0 0 0)
   )
-  (junction (at 234.95 138.43) (diameter 0) (color 0 0 0 0)
-  )
   (junction (at 104.14 39.37) (diameter 0) (color 0 0 0 0)
   )
@@
   (junction (at 78.74 30.48) (diameter 0) (color 0 0 0 0)
   )
-  (junction (at 212.09 139.7) (diameter 0) (color 0 0 0 0)
-  )
   (junction (at 64.77 140.97) (diameter 0) (color 0 0 0 0)
   )
@@
   (no_connect (at 143.51 106.68))
   (no_connect (at 68.58 74.93))
-  (no_connect (at 68.58 62.23))
   (no_connect (at 41.91 158.75))
   (no_connect (at 143.51 86.36))
@@
   (no_connect (at 41.91 173.99))
   (no_connect (at 68.58 67.31))
-  (no_connect (at 68.58 59.69))
   (no_connect (at 143.51 57.15))
+  (no_connect (at 143.51 96.52))
   (no_connect (at 41.91 168.91))
   (no_connect (at 60.96 158.75))
@@
   (no_connect (at 254 38.1))
   (no_connect (at 41.91 163.83))
+  (no_connect (at 143.51 99.06))
   (no_connect (at 68.58 82.55))
   (no_connect (at 143.51 101.6))
@@
   (no_connect (at 175.26 31.75))
   (no_connect (at 143.51 104.14))
-  (no_connect (at 215.9 66.04))
   (no_connect (at 60.96 173.99))
   (no_connect (at 60.96 163.83))
@@
     (stroke (width 0) (type default) (color 0 0 0 0))
   )
-  (wire (pts (xy 254 30.48) (xy 255.27 30.48))
+  (wire (pts (xy 215.9 64.77) (xy 194.31 64.77))
     (stroke (width 0) (type default) (color 0 0 0 0))
   )
-  (wire (pts (xy 220.98 60.96) (xy 220.98 67.31))
+  (wire (pts (xy 254 30.48) (xy 255.27 30.48))
     (stroke (width 0) (type default) (color 0 0 0 0))
   )
-  (wire (pts (xy 212.09 139.7) (xy 212.09 140.97))
+  (wire (pts (xy 220.98 60.96) (xy 220.98 67.31))
     (stroke (width 0) (type default) (color 0 0 0 0))
   )
@@
     (stroke (width 0) (type default) (color 0 0 0 0))
   )
-  (wire (pts (xy 215.9 67.31) (xy 215.9 66.04))
-    (stroke (width 0) (type default) (color 0 0 0 0))
-  )
   (wire (pts (xy 186.69 52.07) (xy 186.69 53.34))
     (stroke (width 0) (type default) (color 0 0 0 0))
@@
     (stroke (width 0) (type default) (color 0 0 0 0))
   )
-  (wire (pts (xy 148.59 96.52) (xy 143.51 96.52))
-    (stroke (width 0) (type default) (color 0 0 0 0))
-  )
   (wire (pts (xy 119.38 29.21) (xy 119.38 30.48))
     (stroke (width 0) (type default) (color 0 0 0 0))
@@
     (stroke (width 0) (type default) (color 0 0 0 0))
   )
+  (wire (pts (xy 66.04 59.69) (xy 68.58 59.69))
+    (stroke (width 0) (type default) (color 0 0 0 0))
+  )
   (wire (pts (xy 168.91 59.69) (xy 168.91 60.96))
     (stroke (width 0) (type default) (color 0 0 0 0))
@@
     (stroke (width 0) (type default) (color 0 0 0 0))
   )
+  (wire (pts (xy 194.31 64.77) (xy 194.31 52.07))
+    (stroke (width 0) (type default) (color 0 0 0 0))
+  )
   (wire (pts (xy 260.35 97.79) (xy 260.35 99.06))
     (stroke (width 0) (type default) (color 0 0 0 0))
@@
     (stroke (width 0) (type default) (color 0 0 0 0))
   )
+  (wire (pts (xy 215.9 67.31) (xy 215.9 64.77))
+    (stroke (width 0) (type default) (color 0 0 0 0))
+  )
   (wire (pts (xy 205.74 33.02) (xy 210.82 33.02))
     (stroke (width 0) (type default) (color 0 0 0 0))
@@
     (stroke (width 0) (type default) (color 0 0 0 0))
   )
+  (wire (pts (xy 66.04 62.23) (xy 68.58 62.23))
+    (stroke (width 0) (type default) (color 0 0 0 0))
+  )
   (wire (pts (xy 44.45 142.24) (xy 44.45 143.51))
     (stroke (width 0) (type default) (color 0 0 0 0))
@@
     (stroke (width 0) (type default) (color 0 0 0 0))
   )
-  (wire (pts (xy 148.59 99.06) (xy 143.51 99.06))
-    (stroke (width 0) (type default) (color 0 0 0 0))
-  )
   (wire (pts (xy 205.74 147.32) (xy 205.74 148.59))
     (stroke (width 0) (type default) (color 0 0 0 0))
   )
-  (wire (pts (xy 234.95 138.43) (xy 234.95 140.97))
-    (stroke (width 0) (type default) (color 0 0 0 0))
-  )
   (wire (pts (xy 171.45 53.34) (xy 186.69 53.34))
     (stroke (width 0) (type default) (color 0 0 0 0))
@@
     )
   )
-  (global_label "XR_TX" (shape input) (at 148.59 99.06 0) (fields_autoplaced)
-    (effects (font (size 1.27 1.27)) (justify left))
-    (property "Intersheet References" "${INTERSHEET_REFS}" (id 0) (at 156.6274 98.9806 0)
-      (effects (font (size 1.27 1.27)) (justify left) hide)
+  (global_label "XR_RX" (shape input) (at 66.04 62.23 180) (fields_autoplaced)
+    (effects (font (size 1.27 1.27)) (justify right))
+    (property "Intersheet References" "${INTERSHEET_REFS}" (id 0) (at 57.7002 62.1506 0)
+      (effects (font (size 1.27 1.27)) (justify right) hide)
     )
   )
@@
     )
   )
-  (global_label "XR_RX" (shape input) (at 148.59 96.52 0) (fields_autoplaced)
-    (effects (font (size 1.27 1.27)) (justify left))
-    (property "Intersheet References" "${INTERSHEET_REFS}" (id 0) (at 156.9298 96.4406 0)
-      (effects (font (size 1.27 1.27)) (justify left) hide)
-    )
-  )
   (global_label "VBUS_PRESENT" (shape input) (at 264.16 88.9 0) (fields_autoplaced)
     (effects (font (size 1.27 1.27)) (justify left))
@@
     )
   )
+  (global_label "XR_TX" (shape input) (at 66.04 59.69 180) (fields_autoplaced)
+    (effects (font (size 1.27 1.27)) (justify right))
+    (property "Intersheet References" "${INTERSHEET_REFS}" (id 0) (at 58.0026 59.6106 0)
+      (effects (font (size 1.27 1.27)) (justify right) hide)
+    )
+  )
   (symbol (lib_id "power:+5V") (at 274.32 25.4 0) (unit 1)
     (in_bom yes) (on_board yes)
@@
     (pin "B9")
   )
-  (symbol (lib_id "Mechanical:MountingHole_Pad") (at 212.09 143.51 180) (unit 1)
-    (in_bom yes) (on_board yes) (fields_autoplaced)
-    (property "Reference" "MH4" (id 0) (at 214.63 143.5099 0)
-      (effects (font (size 1.27 1.27)) (justify right))
-    )
-    (property "Value" "MountingHole_Pad" (id 1) (at 214.63 146.0499 0)
-      (effects (font (size 1.27 1.27)) (justify right))
-    )
-    (property "Footprint" "MountingHole:MountingHole_3mm" (id 2) (at 212.09 143.51 0)
-      (effects (font (size 1.27 1.27)) hide)
-    )
-    (property "Datasheet" "~" (id 3) (at 212.09 143.51 0)
-      (effects (font (size 1.27 1.27)) hide)
-    )
-    (pin "1")
-  )
   (symbol (lib_id "power:+5V") (at 110.49 168.91 0) (unit 1)
     (in_bom yes) (on_board yes)
@@
     (pin "1")
   )
+  (symbol (lib_id "Connector:Conn_01x02_Male") (at 105.41 186.69 0) (unit 1)
+    (in_bom yes) (on_board yes) (fields_autoplaced)
+    (property "Reference" "J5" (id 0) (at 106.045 181.61 0))
+    (property "Value" "Conn_01x02_Male" (id 1) (at 106.045 184.15 0))
+    (property "Footprint" "Connector_PinHeader_2.54mm:PinHeader_1x02_P2.54mm_Vertical" (id 2) (at 105.41 186.69 0)
+      (effects (font (size 1.27 1.27)) hide)
+    )
+    (property "Datasheet" "~" (id 3) (at 105.41 186.69 0)
+      (effects (font (size 1.27 1.27)) hide)
+    )
+    (pin "1")
+    (pin "2")
+  )
   (symbol (lib_id "Device:Crystal") (at 35.56 99.06 270) (unit 1)
     (in_bom yes) (on_board yes)
@@
     (pin "9")
   )
-  (symbol (lib_id "Mechanical:MountingHole_Pad") (at 234.95 143.51 180) (unit 1)
-    (in_bom yes) (on_board yes) (fields_autoplaced)
-    (property "Reference" "MH3" (id 0) (at 237.49 143.5099 0)
-      (effects (font (size 1.27 1.27)) (justify right))
-    )
-    (property "Value" "MountingHole_Pad" (id 1) (at 237.49 146.0499 0)
-      (effects (font (size 1.27 1.27)) (justify right))
-    )
-    (property "Footprint" "MountingHole:MountingHole_3mm" (id 2) (at 234.95 143.51 0)
-      (effects (font (size 1.27 1.27)) hide)
-    )
-    (property "Datasheet" "~" (id 3) (at 234.95 143.51 0)
-      (effects (font (size 1.27 1.27)) hide)
-    )
-    (pin "1")
-  )
   (symbol (lib_id "power:GND1") (at 60.96 52.07 0) (unit 1)
