File: Design/spudglo_driver_v3p1/spudglo_driver_v3p1.kicad_pcb (KiCad board)
At the start: 4 copper layers, 86.3 x 64.6 mm, 117 parts, among them J1 Barrel_Jack_Switch, J10 Conn_01x01_Male, J11 Conn_01x01_Male, J12 Conn_01x01_Male, J13 Conn_01x01_Male, J14 Conn_01x02_Male, J15 Conn_01x01_Male, J16 Conn_01x02_Male, J17 Conn_01x01_Male, J18 Conn_01x08_Male, J19 Conn_01x01_Male, J2 Conn_01x01_Male, J20 Conn_01x01_Male, J21 Conn_01x01_Male, J22 Conn_01x01_Male, J23 Conn_01x01_Male, J24 Conn_01x01_Male, J25 Conn_01x04_Male, J26 Conn_01x04_Male, J27 Conn_01x01_Male, J28 Conn_01x01_Male, J29 Conn_01x04_Male, J3 Conn_01x04_Male, J30 Conn_01x04_Male, J31 Conn_01x04_Male, J33 Conn_01x01_Male, J34 Conn_01x01_Male, J4 Conn_01x01_Male, J5 Conn_01x01_Male, J6 Conn_01x01_Male, J7 Conn_01x01_Male, J8 Conn_01x01_Male, J9 Conn_01x01_Male, Q1 BSS138, Q2 BSS138, SW1 SW_DIP_x01, U1 SN74HCT245PW, U10 receiver_433MHz, U11 receiver_433MHz, U2 STM32L431RCTx, U3 LP5907MFX-3.3, U4 ECS-480-8-36-RWN-TR, U5 receiver_433MHz, U6 ECS-.327-9-1210-TR, U7 PS2501-4, U8 TXB0104D, U9 receiver_433MHz

Commit message: more hw lol
Routing:
- added copper zone on In2.Cu, net +3V3
- added copper zone on In2.Cu, net +5V
- added copper zone on In1.Cu, net GND1
- removed copper zone on PWR.Cu, net +3V3
- removed copper zone on PWR.Cu, net +5V
- removed copper zone on GND.Cu, net GND1
Other:
- net class Default removed
