File: Design/spudglo_driver_v4p3/spudglo_driver_v4p3.kicad_sch (KiCad schematic)
At the start: 22 parts, among them U1 receiver_433MHz, U2 TXS0104EDR, U3 receiver_433MHz, U4 receiver_433MHz, U5 receiver_433MHz, U6 PS2501-4

Commit message: latest hw
Other:
- removed sheet spudglo_v4p2_micro
- added sheet spudglo_v4p3_micro (spudglo_v4p3_micro.kicad_sch)
Changed lines of the file:
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@@
     (pin "1")
     (instances
-      (project "spudglo_driver_v4p2"
+      (project "spudglo_driver_v4p3"
         (path "/52f8bacc-d1b9-4904-87e9-4727c7e9578e"
           (reference "#PWR0104") (unit 1)
@@
     (pin "1")
     (instances
-      (project "spudglo_driver_v4p2"
+      (project "spudglo_driver_v4p3"
         (path "/52f8bacc-d1b9-4904-87e9-4727c7e9578e"
           (reference "#PWR0103") (unit 1)
@@
     (pin "2")
     (instances
-      (project "spudglo_driver_v4p2"
+      (project "spudglo_driver_v4p3"
         (path "/52f8bacc-d1b9-4904-87e9-4727c7e9578e"
           (reference "R24") (unit 1)
@@
     (pin "2")
     (instances
-      (project "spudglo_driver_v4p2"
+      (project "spudglo_driver_v4p3"
         (path "/52f8bacc-d1b9-4904-87e9-4727c7e9578e"
           (reference "R2") (unit 1)
@@
     (pin "2")
     (instances
-      (project "spudglo_driver_v4p2"
+      (project "spudglo_driver_v4p3"
         (path "/52f8bacc-d1b9-4904-87e9-4727c7e9578e"
           (reference "R7") (unit 1)
@@
     (pin "5")
     (instances
-      (project "spudglo_driver_v4p2"
+      (project "spudglo_driver_v4p3"
         (path "/52f8bacc-d1b9-4904-87e9-4727c7e9578e"
           (reference "U4") (unit 1)
@@
     (pin "1")
     (instances
-      (project "spudglo_driver_v4p2"
+      (project "spudglo_driver_v4p3"
         (path "/52f8bacc-d1b9-4904-87e9-4727c7e9578e"
           (reference "#PWR0113") (unit 1)
@@
     (pin "1")
     (instances
-      (project "spudglo_driver_v4p2"
+      (project "spudglo_driver_v4p3"
         (path "/52f8bacc-d1b9-4904-87e9-4727c7e9578e"
           (reference "#PWR0106") (unit 1)
@@
     (pin "9")
     (instances
-      (project "spudglo_driver_v4p2"
+      (project "spudglo_driver_v4p3"
         (path "/52f8bacc-d1b9-4904-87e9-4727c7e9578e"
           (reference "U6") (unit 1)
@@
     (pin "1")
     (instances
-      (project "spudglo_driver_v4p2"
+      (project "spudglo_driver_v4p3"
         (path "/52f8bacc-d1b9-4904-87e9-4727c7e9578e"
           (reference "#PWR0114") (unit 1)
@@
     (pin "2")
     (instances
-      (project "spudglo_driver_v4p2"
+      (project "spudglo_driver_v4p3"
         (path "/52f8bacc-d1b9-4904-87e9-4727c7e9578e"
           (reference "R9") (unit 1)
@@
     (pin "1")
     (instances
-      (project "spudglo_driver_v4p2"
+      (project "spudglo_driver_v4p3"
         (path "/52f8bacc-d1b9-4904-87e9-4727c7e9578e"
           (reference "#PWR0108") (unit 1)
@@
     (pin "2")
     (instances
-      (project "spudglo_driver_v4p2"
+      (project "spudglo_driver_v4p3"
         (path "/52f8bacc-d1b9-4904-87e9-4727c7e9578e"
           (reference "R11") (unit 1)
@@
     (pin "1-UN")
     (instances
-      (project "spudglo_driver_v4p2"
+      (project "spudglo_driver_v4p3"
         (path "/52f8bacc-d1b9-4904-87e9-4727c7e9578e"
           (reference "U2") (unit 1)
@@
     (pin "5")
     (instances
-      (project "spudglo_driver_v4p2"
+      (project "spudglo_driver_v4p3"
         (path "/52f8bacc-d1b9-4904-87e9-4727c7e9578e"
           (reference "U1") (unit 1)
@@
     (pin "2")
     (instances
-      (project "spudglo_driver_v4p2"
+      (project "spudglo_driver_v4p3"
         (path "/52f8bacc-d1b9-4904-87e9-4727c7e9578e"
           (reference "R6") (unit 1)
@@
     (pin "5")
     (instances
-      (project "spudglo_driver_v4p2"
+      (project "spudglo_driver_v4p3"
         (path "/52f8bacc-d1b9-4904-87e9-4727c7e9578e"
           (reference "U5") (unit 1)
@@
     (pin "2")
     (instances
-      (project "spudglo_driver_v4p2"
+      (project "spudglo_driver_v4p3"
         (path "/52f8bacc-d1b9-4904-87e9-4727c7e9578e"
           (reference "R4") (unit 1)
@@
     (pin "1")
     (instances
-      (project "spudglo_driver_v4p2"
+      (project "spudglo_driver_v4p3"
         (path "/52f8bacc-d1b9-4904-87e9-4727c7e9578e"
           (reference "#PWR0112") (unit 1)
@@
     (pin "1")
     (instances
-      (project "spudglo_driver_v4p2"
+      (project "spudglo_driver_v4p3"
         (path "/52f8bacc-d1b9-4904-87e9-4727c7e9578e"
           (reference "#PWR0102") (unit 1)
@@
     (pin "2")
     (instances
-      (project "spudglo_driver_v4p2"
+      (project "spudglo_driver_v4p3"
         (path "/52f8bacc-d1b9-4904-87e9-4727c7e9578e"
           (reference "R12") (unit 1)
@@
     (pin "2")
     (instances
-      (project "spudglo_driver_v4p2"
+      (project "spudglo_driver_v4p3"
         (path "/52f8bacc-d1b9-4904-87e9-4727c7e9578e"
           (reference "R8") (unit 1)
@@
     (pin "1")
     (instances
-      (project "spudglo_driver_v4p2"
+      (project "spudglo_driver_v4p3"
         (path "/52f8bacc-d1b9-4904-87e9-4727c7e9578e"
           (reference "#PWR0115") (unit 1)
@@
     (pin "1")
     (instances
-      (project "spudglo_driver_v4p2"
+      (project "spudglo_driver_v4p3"
         (path "/52f8bacc-d1b9-4904-87e9-4727c7e9578e"
           (reference "#PWR0107") (unit 1)
@@
     (pin "1")
     (instances
-      (project "spudglo_driver_v4p2"
+      (project "spudglo_driver_v4p3"
         (path "/52f8bacc-d1b9-4904-87e9-4727c7e9578e"
           (reference "#PWR0101") (unit 1)
@@
     (pin "2")
     (instances
-      (project "spudglo_driver_v4p2"
+      (project "spudglo_driver_v4p3"
         (path "/52f8bacc-d1b9-4904-87e9-4727c7e9578e"
           (reference "R10") (unit 1)
@@
     (pin "1")
     (instances
-      (project "spudglo_driver_v4p2"
+      (project "spudglo_driver_v4p3"
         (path "/52f8bacc-d1b9-4904-87e9-4727c7e9578e"
           (reference "#PWR0111") (unit 1)
@@
     (pin "2")
     (instances
-      (project "spudglo_driver_v4p2"
+      (project "spudglo_driver_v4p3"
         (path "/52f8bacc-d1b9-4904-87e9-4727c7e9578e"
           (reference "R13") (unit 1)
@@
     (pin "2")
     (instances
-      (project "spudglo_driver_v4p2"
+      (project "spudglo_driver_v4p3"
         (path "/52f8bacc-d1b9-4904-87e9-4727c7e9578e"
           (reference "R1") (unit 1)
@@
     (pin "2")
     (instances
-      (project "spudglo_driver_v4p2"
+      (project "spudglo_driver_v4p3"
         (path "/52f8bacc-d1b9-4904-87e9-4727c7e9578e"
           (reference "R5") (unit 1)
@@
     (pin "1")
     (instances
-      (project "spudglo_driver_v4p2"
+      (project "spudglo_driver_v4p3"
         (path "/52f8bacc-d1b9-4904-87e9-4727c7e9578e"
           (reference "#PWR0116") (unit 1)
@@
     (pin "2")
     (instances
-      (project "spudglo_driver_v4p2"
+      (project "spudglo_driver_v4p3"
         (path "/52f8bacc-d1b9-4904-87e9-4727c7e9578e"
           (reference "C2") (unit 1)
@@
     (pin "1")
     (instances
-      (project "spudglo_driver_v4p2"
+      (project "spudglo_driver_v4p3"
         (path "/52f8bacc-d1b9-4904-87e9-4727c7e9578e"
           (reference "#PWR0105") (unit 1)
@@
     (pin "1")
     (instances
-      (project "spudglo_driver_v4p2"
+      (project "spudglo_driver_v4p3"
         (path "/52f8bacc-d1b9-4904-87e9-4727c7e9578e"
           (reference "#PWR0110") (unit 1)
@@
     (pin "2")
     (instances
-      (project "spudglo_driver_v4p2"
+      (project "spudglo_driver_v4p3"
         (path "/52f8bacc-d1b9-4904-87e9-4727c7e9578e"
           (reference "C1") (unit 1)
@@
     (pin "5")
     (instances
-      (project "spudglo_driver_v4p2"
+      (project "spudglo_driver_v4p3"
         (path "/52f8bacc-d1b9-4904-87e9-4727c7e9578e"
           (reference "U3") (unit 1)
@@
     (pin "1")
     (instances
-      (project "spudglo_driver_v4p2"
+      (project "spudglo_driver_v4p3"
         (path "/52f8bacc-d1b9-4904-87e9-4727c7e9578e"
           (reference "#PWR0109") (unit 1)
@@
     (pin "2")
     (instances
-      (project "spudglo_driver_v4p2"
+      (project "spudglo_driver_v4p3"
         (path "/52f8bacc-d1b9-4904-87e9-4727c7e9578e"
           (reference "R3") (unit 1)
@@
     )
   )
-  (sheet (at 181.61 30.48) (size 40.64 19.05) (fields_autoplaced)
+  (sheet (at 116.84 64.77) (size 19.05 6.35) (fields_autoplaced)
     (stroke (width 0.1524) (type solid))
     (fill (color 0 0 0 0.0000))
-    (property "Sheetname" "spudglo_v4p2_micro" (at 181.61 29.7684 0)
+    (property "Sheetname" "spudglo_v4p3_micro" (at 116.84 64.0584 0)
       (effects (font (size 1.27 1.27)) (justify left bottom))
     )
-    (property "Sheetfile" "spudglo_v4p2_micro.kicad_sch" (at 181.61 50.1146 0)
+    (property "Sheetfile" "spudglo_v4p3_micro.kicad_sch" (at 116.84 71.7046 0)
       (effects (font (size 1.27 1.27)) (justify left top))
     )
     (instances
-      (project "spudglo_driver_v4p2"
-        (path "/52f8bacc-d1b9-4904-87e9-4727c7e9578e" (page "2"))
-      )
-    )
+      (project "spudglo_driver_v4p3"
+        (path "/52f8bacc-d1b9-4904-87e9-4727c7e9578e" (page "3"))
+      )
+    )
