File: Design/spudglo_driver_v4p3/spudglo_v4p3_micro.kicad_sch (KiCad schematic)
At the start: 59 parts, among them J1 Conn_01x08_Male, J2 Barrel_Jack_Switch, J3 terminal_custom_12pin, J4 Conn_01x08_Male, J5 Conn_01x02_Male, U10 STM32L431RCTx, U11 LP5907MFX-3.3, U12 USB-C-31-M-12, U13 XR21B1411, U14 NCP361, U7 ECS-.327-9-1210-TR, U8 ECS-480-8-36-RWN-TR, U9 SN74HCT245PW

Commit message: latest hw
Parts:
- removed J5: Conn_01x02_Male, Connector_PinHeader_2.54mm:PinHeader_1x02_P2.54mm_Vertical, symbol Connector:Conn_01x02_Male
- added D1: GREEN LED, LED_SMD:LED_0402_1005Metric_Pad0.77x0.64mm_HandSolder, symbol Device:LED
- added D3: RED_LED, LED_SMD:LED_0402_1005Metric_Pad0.77x0.64mm_HandSolder, symbol Device:LED
- added R37, R39: 1k, Resistor_SMD:R_0402_1005Metric, symbol Device:R
- R25, R26: value 5.1k -> DNI
Connections:
- net +3V3: now also U12.A8 (SBU1)
- net GND1: now also R37.2, R39.2
- net NRST: now also U12.B8 (SBU2)
- net SWCLK: now also R25.1, U12.B5 (CC2)
- net SWDIO: now also R26.1, U12.A5 (CC1)
- net GREEN_LED: now reaches U10.10 (PC2/SPI2_MISO)
- net GREEN_LED: now also D1.2 (A)
- net RED_LED: now reaches U10.11 (PC3/SPI2_MOSI)
- net RED_LED: now also D3.2 (A)
- new net: D3.1 (K), R37.1
- new net: D1.1 (K), R39.1
- no-connect marks 37 -> 33
Other:
- moved on the sheet: R33

Commit message: spudglo v6 added
Parts:
- added D2: BLUE LED, LED_SMD:LED_0603_1608Metric, symbol Device:LED
- added D4: ORANGE LED, LED_SMD:LED_0603_1608Metric, symbol Device:LED
- added R38, R40: 100, Resistor_SMD:R_0402_1005Metric, symbol Device:R
- D1, D3: footprint LED_SMD:LED_0402_1005Metric_Pad0.77x0.64mm_HandSolder -> LED_SMD:LED_0603_1608Metric
- R37, R39: value 1k -> 100
Connections:
- net GND1: now also R38.2, R40.2
- net BLUE_LED: now reaches U10.61 (PB8/I2C1_SCL/TIM16_CH1)
- net BLUE_LED: now also D2.2 (A)
- net ORANGE_LED: now reaches U10.62 (PB9/I2C1_SDA/SPI2_NSS)
- net ORANGE_LED: now also D4.2 (A)
- new net: D4.1 (K), R38.1
- new net: D2.1 (K), R40.1
- no-connect marks 33 -> 31
