File: Design/usb_programmer/usb_programmer.kicad_sch (KiCad schematic)
At the start: 24 parts, among them J1 Conn_01x20_Male, J2 Conn_01x02_Pin, J3 Conn_01x02_Pin, J5 Conn_01x02_Male, J6 Conn_01x02_Male, P1 USB_C_Plug, Q2 BSS138, Q3 BSS138, U1 USB-C-31-M-12

Commit message: spudglo v6 added
Parts:
- removed J1: Conn_01x20_Male, Connector_PinHeader_2.54mm:PinHeader_2x10_P2.54mm_Vertical, symbol programmer_adapter_v2-rescue:Conn_01x20_Male-Connector
- removed J3: Conn_01x02_Pin, Connector_PinHeader_2.54mm:PinHeader_1x02_P2.54mm_Vertical, symbol Connector:Conn_01x02_Pin
- removed MH1, MH2: MountingHole_Pad, MountingHole:MountingHole_3mm, symbol Mechanical:MountingHole_Pad
- removed R1: 0, Resistor_SMD:R_0402_1005Metric, symbol Device:R
- added J1: Conn_01x08_Male, Connector_PinHeader_2.54mm:PinHeader_2x04_P2.54mm_Vertical, symbol Connector:Conn_01x08_Male
Connections:
- net GND1: now also J1.1 (Pin_1)
- net NRST: now also J1.2 (Pin_2)
- net SWCLK: now also J1.6 (Pin_6)
- net SWDIO: now also J1.7 (Pin_7)
- new net +3V3: J1.8 (Pin_8)
- no-connect marks 17 -> 15
