File: Design/mn_wild_siren_rpi/Untitled/mn_wild_siren_micro.kicad_sch (KiCad schematic)
At the start: 52 parts, among them J1 Barrel_Jack_Switch, J10 Conn_01x16_Male, J13 Conn_01x03_Male, J14 Conn_01x03_Male, J20 Conn_01x40_Male, J22 Conn_01x02_Male, J239 Conn_01x02_Male, J3 Conn_01x04_Male, Q3 BSS138, Q4 BSS138, U2 SN74HCT245PW, U4 TXS0104EDR, U5 TLV75733PDBV, U6 SN74HCT245PW

Commit message: add bus_bar, led_dog_collar, mn_wild_siren_2.0
Parts:
- removed C10, C4: 0.1u, Capacitor_SMD:C_0402_1005Metric, symbol Device:C_Small
- removed C11, C5, C6, C8: 0.1u, Capacitor_SMD:C_0603_1608Metric, symbol Device:C_Small
- removed C12, C20, C22, C23, C25, C7, C9: 1u, Capacitor_SMD:C_0603_1608Metric, symbol Device:C_Small
- removed C14, C17: 10u, Capacitor_SMD:C_0603_1608Metric_Pad1.08x0.95mm_HandSolder, symbol spudglo_driver_v3p1-rescue:CP_Small-Device
- removed C15, C16, C18, C19: 1u, Capacitor_SMD:C_0603_1608Metric_Pad1.08x0.95mm_HandSolder, symbol spudglo_driver_v3p1-rescue:CP_Small-Device
- removed C2, C3: 1u, Capacitor_SMD:C_0603_1608Metric_Pad1.08x0.95mm_HandSolder, symbol Device:C_Small
- removed C21, C24: 10u, Capacitor_SMD:C_0603_1608Metric, symbol Device:C_Small
- removed F1: Fuse-2410FA, srw_custom:2410FA, symbol srw_custom:Fuse-2410FA
- removed H1, H2, H3, H4: MountingHole, MountingHole:MountingHole_3.2mm_M3, symbol Mechanical:MountingHole
- removed J1: Barrel_Jack_Switch, Connector_BarrelJack:BarrelJack_Wuerth_6941xx301002, symbol Connector:Barrel_Jack_Switch
- removed J10: Conn_01x16_Male, Connector_PinHeader_2.54mm:PinHeader_2x08_P2.54mm_Vertical, symbol Connector:Conn_01x16_Male
- removed J13: Conn_01x03_Male, srw_custom:1984620, symbol Connector:Conn_01x03_Male
- removed J14: Conn_01x03_Male, Connector_PinHeader_2.54mm:PinHeader_1x03_P2.54mm_Vertical, symbol Connector:Conn_01x03_Male
- removed J20: Conn_01x40_Male, Connector_PinHeader_2.54mm:PinHeader_2x20_P2.54mm_Vertical, symbol Connector:Conn_01x40_Male
- removed J22, J239: Conn_01x02_Male, Connector_PinHeader_2.54mm:PinHeader_1x02_P2.54mm_Vertical, symbol Connector:Conn_01x02_Male
- removed J3: Conn_01x04_Male, srw_custom:1984633, symbol Connector:Conn_01x04_Male
- removed Q3, Q4: BSS138, Package_TO_SOT_SMD:SOT-23, symbol Transistor_FET:BSS138
- removed R11: 1M, Resistor_SMD:R_0402_1005Metric, symbol Device:R
- removed R15: 1M, Resistor_SMD:R_0603_1608Metric_Pad0.98x0.95mm_HandSolder, symbol Device:R
- removed R21, R22, R26: DNI, Resistor_SMD:R_0402_1005Metric, symbol Device:R
- removed R25: 0, Resistor_SMD:R_0402_1005Metric, symbol Device:R
- removed R36, R37: 10k, Resistor_SMD:R_0402_1005Metric, symbol Device:R
- removed R388, R399: 1k, Resistor_SMD:R_0402_1005Metric, symbol Device:R
- removed U2, U6: SN74HCT245PW, Package_SO:TSSOP-20_4.4x6.5mm_P0.65mm, symbol srw_custom:SN74HCT245PW
- removed U4: TXS0104EDR, Package_SO:SOIC-14_3.9x8.7mm_P1.27mm, symbol srw_custom:TXS0104EDR
- removed U5: TLV75733PDBV, Package_TO_SOT_SMD:SOT-23-5, symbol Regulator_Linear:TLV75733PDBV
Connections:
- no-connect marks 9 -> 0
