File: Design/mn_wild_siren_rpi/Untitled/mn_wild_siren_micro_v2p0.kicad_sch (KiCad schematic)
At the start: 61 parts, among them J1 Barrel_Jack_Switch, J10 Conn_01x16_Male, J13 Conn_01x03_Male, J14 Conn_01x03_Male, J20 Conn_01x40_Male, J22 Conn_01x02_Male, J239 Conn_01x02_Male, J3 Conn_01x04_Male, Q3 BSS138, Q4 BSS138, U2 SN74HCT245PW, U3 rf_433MHz_module, U4 RV-8803, U5 TLV75733PDBV, U6 SN74HCT245PW, U7 rf_433MHz_module

Commit message: add spudglo v8p0
Other:
- note added: "GPIO0"
- note added: "GPIO1"
- note added: "GPIO10"
- note added: "GPIO11"
- note added: "GPIO12"
- note added: "GPIO13"
- note added: "GPIO14"
- note added: "GPIO15"
- note added: "GPIO16"
- note added: "GPIO17"
- note added: "GPIO18"
- note added: "GPIO19"
- note added: "GPIO2"
- note added: "GPIO20"
- note added: "GPIO21"
- note added: "GPIO22"
- note added: "GPIO23"
- note added: "GPIO24"
- note added: "GPIO25"
- note added: "GPIO26"
- note added: "GPIO27"
- note added: "GPIO3"
- note added: "GPIO4"
- note added: "GPIO5"
- note added: "GPIO6"
- note added: "GPIO7"
- note added: "GPIO8"
- note added: "GPIO9"
