File: Design/led_dog_collar/led_dog_collar.kicad_pcb (KiCad board)
At the start: 4 copper layers, 31.7 x 25 mm, 54 parts, among them J1 Conn_01x02_Socket, J2 Conn_01x01_Male, J3 Conn_01x08_Male, J4 Conn_01x01_Male, J5 Conn_01x01_Male, SW2 EG1206A, U2 SN74HCT245PW, U3 LP5907MFX-3.3, U4 STM32L431RCTx, U5 ECS-480-8-36-RWN-TR, U6 ECS-.327-9-1210-TR

Commit message: add spudglo v8p0
Connections:
- SW2 pad 1: VBAT -> unconnected-(SW2-Pad1)
- SW2 pad 2: unconnected-(SW2-Pad2) -> VBAT
Routing:
- net VBAT: track 43.9 -> 42.1 mm
Changed lines of the file:
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@@
 	(net 60 "Net-(U1-IND)")
 	(net 61 "VBAT")
-	(net 62 "unconnected-(SW2-Pad2)")
+	(net 62 "unconnected-(SW2-Pad1)")
 	(net 63 "unconnected-(J3-Pin_3-Pad3)")
 	(net 64 "unconnected-(J3-Pin_4-Pad4)")
@@
 			(layers "*.Cu" "*.Mask")
 			(remove_unused_layers no)
-			(net 61 "VBAT")
+			(net 62 "unconnected-(SW2-Pad1)")
 			(pinfunction "1")
-			(pintype "unspecified")
+			(pintype "unspecified+no_connect")
 		)
 		(pad "2" thru_hole circle
@@
 			(layers "*.Cu" "*.Mask")
 			(remove_unused_layers no)
-			(net 62 "unconnected-(SW2-Pad2)")
+			(net 61 "VBAT")
 			(pinfunction "2")
-			(pintype "unspecified+no_connect")
+			(pintype "unspecified")
 		)
 		(pad "3" thru_hole circle
@@
 	)
 	(gr_text "VBAT_EN"
-		(at 182.78 64.4 0)
+		(at 182.95 64.33 0)
 		(layer "B.SilkS")
 		(effects
@@
 	)
 	(gr_text "VBAT"
-		(at 182.1 58.4 0)
+		(at 182.31 61.18 0)
 		(layer "B.SilkS")
 		(effects
@@
 		)
 	)
-	(gr_text "ON"
-		(at 181.26 53.65 0)
+	(gr_text "GND"
+		(at 205.54 71.34 -135)
 		(layer "B.SilkS")
 		(effects
@@
 				(thickness 0.125)
 			)
-			(justify mirror)
 		)
 	)
-	(gr_text "GND"
-		(at 205.54 71.34 -135)
+	(gr_text "ON"
+		(at 182.88 68.48 -0)
 		(layer "B.SilkS")
 		(effects
@@
 				(thickness 0.125)
 			)
+			(justify mirror)
 		)
 	)
 	(gr_text "NC"
-		(at 182.02 61.25 0)
+		(at 181.88 58.26 0)
 		(layer "B.SilkS")
 		(effects
@@
 	)
 	(gr_text "OFF"
-		(at 183.25 68.4 0)
+		(at 181.42 53.61 0)
 		(layer "B.SilkS")
 		(effects
@@
 	)
 	(gr_text "OFF"
-		(at 183.23 68.49 0)
+		(at 181.39 53.6 0)
 		(layer "F.SilkS")
 		(effects
@@
 	)
 	(gr_text "ON"
-		(at 178.74 53.53 0)
+		(at 182.9 68.48 0)
 		(layer "F.SilkS")
 		(effects
@@
 	)
 	(segment
-		(start 180.104601 58.27)
-		(end 180.086 58.288601)
+		(start 178.9375 62.4371)
+		(end 180.086 61.2886)
 		(width 0.5)
 		(layer "F.Cu")
@@
 	)
 	(segment
-		(start 178.9375 64.764324)
-		(end 180.373176 66.2)
+		(start 183.82 58.27)
+		(end 183.1046 58.27)
 		(width 0.5)
 		(layer "F.Cu")
@@
 	)
 	(segment
-		(start 180.086 58.288601)
-		(end 178.9375 59.437101)
+		(start 178.9375 64.764324)
+		(end 178.9375 62.4371)
 		(width 0.5)
 		(layer "F.Cu")
@@
 	)
 	(segment
-		(start 200.819999 70.78)
-		(end 199.82 70.78)
+		(start 178.9375 64.764324)
+		(end 180.373176 66.2)
 		(width 0.5)
 		(layer "F.Cu")
@@
 	)
 	(segment
-		(start 183.82 58.27)
-		(end 180.104601 58.27)
+		(start 200.819999 70.78)
+		(end 199.82 70.78)
 		(width 0.5)
 		(layer "F.Cu")
@@
 	)
 	(segment
-		(start 178.9375 59.437101)
-		(end 178.9375 64.764324)
+		(start 198.83 70.78)
+		(end 199.82 70.78)
 		(width 0.5)
 		(layer "F.Cu")
@@
 	)
 	(segment
-		(start 198.83 70.78)
-		(end 199.82 70.78)
+		(start 200.819999 70.78)
+		(end 200.819999 72.915801)
 		(width 0.5)
 		(layer "F.Cu")
@@
 	)
 	(segment
-		(start 200.819999 70.78)
-		(end 200.819999 72.915801)
+		(start 183.1046 58.27)
+		(end 180.086 61.2886)
 		(width 0.5)
 		(layer "F.Cu")
@@
 		(net 61)
 	)
+	(segment
+		(start 180.104601 58.27)
+		(end 180.086 58.288601)
+		(width 0.5)
+		(layer "F.Cu")
+		(net 62)
+	)
 	(zone
