File: Design/led_dog_collar/led_dog_collar.kicad_sch (KiCad schematic)
At the start: 45 parts, among them J1 Conn_01x02_Socket, J2 Conn_01x01_Male, J3 Conn_01x08_Male, J4 Conn_01x01_Male, J5 Conn_01x01_Male, SW2 EG1206A, U2 SN74HCT245PW, U3 LP5907MFX-3.3, U4 STM32L431RCTx, U5 ECS-480-8-36-RWN-TR, U6 ECS-.327-9-1210-TR

Commit message: add spudglo v8p0
Connections:
- net VBAT: now also SW2.2; no longer SW2.1
Changed lines of the file:
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@@
+	)
+	(no_connect
+		(at 233.68 95.25)
 	)
 	(no_connect
@@
 	)
 	(no_connect
-		(at 259.08 97.79)
-	)
-	(no_connect
 		(at 134.62 64.77)
 	)
@@
 	(wire
 		(pts
+			(xy 259.08 101.6) (xy 260.35 101.6)
+		)
+		(stroke
+			(width 0)
+			(type default)
+		)
+	)
+	(wire
+		(pts
 			(xy 266.7 135.89) (xy 266.7 142.24)
 		)
@@
 	(wire
 		(pts
+			(xy 259.08 97.79) (xy 260.35 97.79)
+		)
+		(stroke
+			(width 0)
+			(type default)
+		)
+	)
+	(wire
+		(pts
 			(xy 266.7 130.81) (xy 266.7 129.54)
 		)
@@
 	(wire
 		(pts
-			(xy 232.41 95.25) (xy 233.68 95.25)
-		)
-		(stroke
-			(width 0)
-			(type default)
-		)
-	)
-	(wire
-		(pts
 			(xy 245.11 129.54) (xy 242.57 129.54)
 		)
@@
 		(pts
 			(xy 92.71 26.67) (xy 92.71 24.13)
+		)
+		(stroke
+			(width 0)
+			(type default)
+		)
+	)
+	(wire
+		(pts
+			(xy 260.35 97.79) (xy 260.35 101.6)
 		)
 		(stroke
@@
 		)
 	)
-	(label "VBAT"
-		(at 232.41 95.25 180)
-		(fields_autoplaced yes)
-		(effects
-			(font
-				(size 1.27 1.27)
-			)
-			(justify right bottom)
-		)
-	)
 	(label "5V_EN"
 		(at 242.57 40.64 180)
@@
 		)
 	)
+	(label "VBAT"
+		(at 259.08 101.6 180)
+		(fields_autoplaced yes)
+		(effects
+			(font
+				(size 1.27 1.27)
+			)
+			(justify right bottom)
+		)
+	)
