File: Design/spud_glo_mini/spud_glo_mini.kicad_pcb (KiCad board)
At the start: 4 copper layers, 36.1 x 29.2 mm, 60 parts, among them J1 Barrel_Jack_Switch, J2 Conn_01x03_Male, U1 TXS0104EDR, U10 XR21B1411, U11 NCP361, U2 PS2501L-1, U3 receiver_433MHz, U4 ECS-.327-9-1210-TR, U5 ECS-480-8-36-RWN-TR, U6 SN74HCT245PW, U7 STM32L431RCTx, U8 LP5907MFX-3.3, U9 USB-C-31-M-12

Commit message: add spudglo v8p0
Parts:
- removed the G*** at (157.6, 113.8)
