File: Design/spudglo_business_card/spudglo_business_card/spudglo_business_card_micro.kicad_sch (KiCad schematic)
At the start: 90 parts, among them J1 Conn_01x08_Male, U10 STM32L431RCTx, U11 LP5907MFX-3.3, U7 ECS-.327-9-1210-TR, U8 ECS-480-8-36-RWN-TR, U9 SN74HCT245PW

Commit message: add spudglo v8p0
Parts:
- renumbered C2 to C25, C2 to C26, C2 to C27, C2 to C28, C2 to C29, C2 to C30, C2 to C31, C2 to C32, C2 to C33, C2 to C34, C2 to C35, C2 to C36, C2 to C37, C2 to C38, C2 to C39, C2 to C40, C2 to C41, C2 to C42, C2 to C43, C2 to C44, C2 to C45, C2 to C46, C2 to C47, C2 to C48, C2 to C49, C2 to C50, C2 to C51, C2 to C52, C2 to C53, C2 to C54, C2 to C55, C2 to C56, C2 to C57, C2 to C58, C2 to C59, C2 to C60, C2 to C61, C2 to C62, C2 to C63, C2 to C64, C2 to C65, C2 to C66, C2 to C67, C2 to C68, C2 to C69, C2 to C70
