File: Design/spudglo_driver_v8p0/spudglo_v8p0_power.kicad_sch (KiCad schematic)
At the start: 27 parts, among them IC1 AP63205, J2 Barrel_Jack_Switch, J4 Conn_01x01_Pin, J5 Conn_01x01_Pin, U14 LP5907MFX-3.3, U16 TPS22916BYFPT

Commit message: add new spudglo boards
Parts:
- added BT1: Battery_Cell, Battery:BatteryHolder_Keystone_500, symbol Device:Battery_Cell
- added C12: 10u, Capacitor_SMD:C_0402_1005Metric_Pad0.74x0.62mm_HandSolder, symbol spudglo_driver_v3p1-rescue:CP_Small-Device
- added R18, R19: DNI, Resistor_SMD:R_0402_1005Metric_Pad0.72x0.64mm_HandSolder, symbol Device:R
Connections:
- net GND1: now also BT1.2 (-), C12.2
- net VIN: now also R19.1
- net at C18.1, R24.1, U17.6 (VOUT): now also R19.2
- net at C28.1, R6.2, R7.1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: now also C12.1
- net at C24.1, C27.1, C30.1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: now also R18.1
- net at C31.1, R9.1, U16.A1 (VOUT): now also R18.2
- new net V_BUTTON: BT1.1 (+)
Other:
- note added: "POWER STEPS VIN == 5 V * MIC826 * N_RESET [5V_BUCK_EN_N] = 0 * RESET [5V_BUCK_BYPASS] = ~ 5 * 2/5 = 2 V * ADP63205 * OFF! * TPS22916B * OFF! * TPS22810 * ON! * VIN CONNECTS TO 5V RAIL VIN == 12 V * MIC826 * N_RESET [5V_BUCK_EN_N] = 4.8 V * RESET [5V_BUCK_BYPASS] = 0 * ADP63205 * ON! * 5V GENERATED * TPS22916B * ON! * ADP 5V CONNECTS TO 5V RAIL. * TPS22810 * OFF! * VIN CONNECTS TO 5V RAIL"
- moved on the sheet: R6
