File: Design/spudglo_driver_v8p0/spudglo_v8p0_power.kicad_sch (KiCad schematic)
At the start: 31 parts, among them IC1 AP63205, J2 Barrel_Jack_Switch, J4 Conn_01x01_Pin, J5 Conn_01x01_Pin, U14 LP5907MFX-3.3, U16 TPS22916BYFPT, U17 TPS22810TDBVRQ1, U7 MIC826SYMT

Commit message: khg
Parts:
- removed BT1: Battery_Cell, Battery:BatteryHolder_Keystone_500, symbol Device:Battery_Cell
- removed C12: 10u, Capacitor_SMD:C_0402_1005Metric_Pad0.74x0.62mm_HandSolder, symbol spudglo_driver_v3p1-rescue:CP_Small-Device
- removed C30, C31: 1u, Capacitor_SMD:C_0402_1005Metric_Pad0.74x0.62mm_HandSolder, symbol spudglo_driver_v3p1-rescue:CP_Small-Device
- removed F1: Fuse-2410FA, srw_custom:2410FA, symbol srw_custom:Fuse-2410FA
- removed J2: Barrel_Jack_Switch, Connector_BarrelJack:BarrelJack_Wuerth_6941xx301002, symbol Connector:Barrel_Jack_Switch
- removed J4, J5: Conn_01x01_Pin, Connector_Pin:Pin_D1.3mm_L11.0mm_LooseFit, symbol Connector:Conn_01x01_Pin
- removed R11, R8: 10k, Resistor_SMD:R_0402_1005Metric_Pad0.72x0.64mm_HandSolder, symbol Device:R
- removed R7: 39k, Resistor_SMD:R_0402_1005Metric_Pad0.72x0.64mm_HandSolder, symbol Device:R
- removed U7: MIC826SYMT, srw_custom:MIC826SYMT, symbol srw_custom:MIC826SYMT
- added C17: 22u, Capacitor_SMD:C_0402_1005Metric_Pad0.74x0.62mm_HandSolder, symbol spudglo_driver_v3p1-rescue:CP_Small-Device
- added U11: MMSZ5244BT1G, srw_custom:SOD-123_ONS, symbol srw_custom:MMSZ5244BT1G
- C27: value 22u -> 1u
- C28: value 0.1u -> 1u
- C5: value 10u -> 0.1u
- L1: value L -> 4.7 uH
- R18: value DNI -> 0
- R6: value 62k -> 100k
- R9: value 0 -> DNI
- U16: value TPS22916BYFPT -> TPS22916CNYFPT; footprint srw_custom:TPS22916BYFPT -> srw_custom:TPS22916CNYFPT; AVAILABILITY Unavailable -> (none); Availability In Stock -> (none); Check_prices https://www.snapeda.com/parts/TPS22916BYFPT/Texas+Instrumen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 -> (none); Description_1 5.5-V, 2-A, 60-mΩ, 10-nA leakage load switch with output di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 -> (none); MP TPS22916BYFPT -> (none); PRICE 0.42 USD -> (none); Price None -> (none); SnapEDA_Link https://www.snapeda.com/parts/TPS22916BYFPT/Texas+Instrumen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 -> (none)
Connections:
- net +5V: now also R18.2, R6.2; no longer R9.2
- net GND1: now also R6.1, C17.2, U11.2 (ANODE)
- net at C28.1: now also R18.1, R9.2, U16.A1 (VOUT); no longer R6.2
- net at C24.1, C27.1, IC1.1 (FB)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: now also R9.1, C17.1; no longer R18.1
- net VIN renamed VIN_LIM
- net VIN_LIM: now also U11.1 (CATHODE); no longer R6.1
- no-connect marks 4 -> 2
Other:
- note added: "VIN_UV = VUV_LO[R] * (R1 + R2 + R3) / (R2 + R3) VIN_UV = 1.2 * (768000 + 226000 + 100000) / (226000 + 100000) VIN_UV = 13.13 V VIN_OV = VOV_R * (R1 + R2 + R3) / (R3) VIN_OV = 1.2 * (768000 + 226000 + 100000) / (100000) VIN_OV = 4.03 V"
- note removed: "Input power"
- note removed: "MIC826TYMT-TR"
- note removed: "MIC826TYMT-TR * Threshold voltage 3.085 V typ * VCC min = 1 V. VCC max = 5.5 V * If VIN = 5 V, VCC = 2 V * N_RST_OUT = 0 * RST_OUT >= 0.8 * 2 V >= 1.6 V * If VIN = 12 V, VCC = 4.8 V * N_RST_OUT = 4.8 V * RST_OUT = 0"
- note removed: "POWER STEPS VIN == 5 V * MIC826 * N_RESET [5V_BUCK_EN_N] = 0 * RESET [5V_BUCK_BYPASS] = ~ 5 * 2/5 = 2 V * ADP63205 * OFF! * TPS22916B * OFF! * TPS22810 * ON! * VIN CONNECTS TO 5V RAIL VIN == 12 V * MIC826 * N_RESET [5V_BUCK_EN_N] = 4.8 V * RESET [5V_BUCK_BYPASS] = 0 * ADP63205 * ON! * 5V GENERATED * TPS22916B * ON! * ADP 5V CONNECTS TO 5V RAIL. * TPS22810 * OFF! * VIN CONNECTS TO 5V RAIL"
- note removed: "VIN select control"
- moved on the sheet: C18, C25, C29, C32, R19, R24, U14, U17
