File: Design/spudglo_driver_v8p0/spudglo_driver_v8p0.kicad_pcb (KiCad board)
At the start: 4 copper layers, 74 x 44 mm, 95 parts, among them J1 Conn_01x01_Pin, J10 Conn_01x01_Pin, J12 1935174, J13 1935174, J14 1935174, J2 1935161, J5 Conn_01x08_Male, J8 Conn_01x01_Pin, J9 Conn_01x01_Pin, U1 rf_433MHz_module, U2 rf_433MHz_module, U3 rf_433MHz_module, U4 rf_433MHz_module, U5 TPS7A2033PDBVR, U7 TPS561201DDCR, U8 STM32L431RCTx, U9 SN74HCT245PW, Y1 ECS-480-8-36-RWN-TR

Commit message: latest hw
Parts:
- added G***: LOGO, LOGO, B.Cu at (169.9, 137.3)
- added G***: LOGO, LOGO, B.Cu at (128.0, 136.3)
- added G***: LOGO, LOGO, F.Cu at (196.3, 163.4)
- moved G*** 0.66 mm to (128.3, 136.5)
